Commit message: Added missing hokuyo.gazebo.xacro file

File: urdfs/sensors/hokuyo_laser.urdf.xacro (robot description, xacro)
@@ -1,4 +1,6 @@
 <?xml version="1.0"?>
 <robot xmlns:xacro="http://ros.org/wiki/xacro">
+	<!-- dima -->
+	<xacro:include filename="$(find sensors_description)/urdfs/sensors/hokuyo_laser.gazebo.xacro" />
 	<xacro:macro name="hokuyo_laser" params="name parent *origin ros_topic update_rate min_angle max_angle range">
 		<joint name="${name}_joint" type="fixed">
@@ -10,5 +12,5 @@
 		<!-- go from the base of the laser to the actual sensor location -->
 		<joint name="${name}_laser_joint" type="fixed">
-			<origin xyz="0 0 0.058" />
+			<origin xyz="0 0 0.058" rpy="0 0 0"/>
 			<parent link="${name}_mount_link"/>
 			<child link="${name}"/>
@@ -36,5 +38,5 @@
 		</link>
 		<!-- gazebo extensions -->
-		<xacro:hokuyo_laser_gazebo name="${name}_laser" ros_topic="${ros_topic}" update_rate="${update_rate}" min_angle="${min_angle}" max_angle="${max_angle}" range="${range}"/>
+		<xacro:hokuyo_laser_gazebo link_name="${name}" frame_name="${name}" ros_topic="${ros_topic}" update_rate="${update_rate}" min_angle="${min_angle}" max_angle="${max_angle}" range="${range}"/>
     </xacro:macro>
 </robot>
