Commit message: [bugfix] Now the Multisense urdf works in the robot

File: urdfs/sensors/multisense_sl.gazebo.xacro (robot description, xacro)
@@ -10,16 +10,16 @@
 			<mu2>0.9</mu2>
 		</gazebo>
-		<gazebo reference="hokuyo_link">
+		<gazebo reference="${prefix}/hokuyo_link">
 			<mu1>0.9</mu1>
 			<mu2>0.9</mu2>
 		</gazebo>
-		<gazebo reference="head_hokuyo_frame">
+		<gazebo reference="${prefix}/head_hokuyo_frame">
 			<mu1>0.9</mu1>
 			<mu2>0.9</mu2>
 		</gazebo>
-		<gazebo reference="hokuyo_joint">
+		<gazebo reference="${prefix}/head_hokuyo_frame_joint">
 			<implicitSpringDamper>1</implicitSpringDamper>
 		</gazebo>
-		<gazebo reference="head_hokuyo_frame">
+		<gazebo reference="${prefix}/head_hokuyo_frame">
 			<sensor type="gpu_ray" name="head_hokuyo_sensor">
 				<pose>0 0 0 0 0 0</pose>
@@ -50,12 +50,12 @@
 					</noise>
 				</ray>
-				<plugin name="gazebo_ros_head_hokuyo_controller" filename="libgazebo_ros_gpu_laser.so">
-					<topicName>/multisense/lidar_scan</topicName>
-					<frameName>head_hokuyo_frame</frameName>
+				<plugin name="${prefix}/head_hokuyo_controller" filename="libgazebo_ros_gpu_laser.so">
+					<topicName>${prefix}/lidar_scan</topicName>
+					<frameName>${prefix}/head_hokuyo_frame</frameName>
 				</plugin>
 			</sensor>
 		</gazebo>
-		<gazebo reference="left_camera_frame">
-			<sensor type="multicamera" name="stereo_camera">
+		<gazebo reference="${prefix}/left_camera_frame">
+			<sensor type="multicamera" name="${prefix}/stereo_camera">
 			<!-- see MultiSenseSLPlugin.h for available modes -->
 			<update_rate>10.0</update_rate>
@@ -111,11 +111,11 @@
 				</noise>
 			</camera>
-			<plugin name="stereo_camera_controller" filename="libgazebo_ros_multicamera.so">
+			<plugin name="${prefix}/stereo_camera_controller" filename="libgazebo_ros_multicamera.so">
 				<alwaysOn>true</alwaysOn>
 				<updateRate>0.0</updateRate>
-				<cameraName>multisense/camera</cameraName>
-				<imageTopicName>image_raw</imageTopicName>
+				<cameraName>${prefix}/camera</cameraName>
+				<imageTopicName>image_color</imageTopicName>
 				<cameraInfoTopicName>camera_info</cameraInfoTopicName>
-				<frameName>left_camera_optical_frame</frameName>
+				<frameName>${prefix}/left_camera_optical_frame</frameName>
 				<!--<rightFrameName>right_camera_optical_frame</rightFrameName>-->
 				<hackBaseline>0.07</hackBaseline>
@@ -128,9 +128,9 @@
 			</sensor>
 		</gazebo>
-		<gazebo reference="head_imu_link">
+		<gazebo reference="${prefix}/head_imu_link">
 			<!-- this is expected to be reparented to head with appropriate offset
 			when head_imu_link is reduced by fixed joint reduction -->
 			<!-- todo: this is working with gazebo 1.4, need to write a unit test -->
-			<sensor name="head_imu_sensor" type="imu">
+			<sensor name="${prefix}/head_imu_sensor" type="imu">
 				<always_on>1</always_on>
 				<update_rate>1000.0</update_rate>
@@ -173,10 +173,10 @@
 			<plugin filename="libMultiSenseSLPlugin.so" name="multisense_plugin"/>
 		</gazebo>
-		<transmission name="hokuyo_trans">
+		<transmission name="${prefix}/hokuyo_trans">
 			<type>transmission_interface/SimpleTransmission</type>
-			<joint name="hokuyo_joint">
+			<joint name="${prefix}/hokuyo_joint">
 				<hardwareInterface>EffortJointInterface</hardwareInterface>
 			</joint>
-			<actuator name="hokuyo_motor">
+			<actuator name="${prefix}/hokuyo_motor">
 				<hardwareInterface>EffortJointInterface</hardwareInterface>
 				<mechanicalReduction>1</mechanicalReduction>

File: urdfs/sensors/multisense_sl.urdf.xacro (robot description, xacro)
@@ -1,5 +1,4 @@
 <?xml version="1.0" ?>
 <robot xmlns:xacro="http://ros.org/wiki/xacro">
-<xacro:include filename="$(find sensors_description)/urdfs/sensors/multisense_sl.gazebo.xacro"/>
 <xacro:macro name="multisense_sl" params="parent *origin prefix" >
   <joint name="${parent}_head_root_joint" type="fixed">
@@ -36,36 +35,27 @@
   </collision>
   </link>
-  <joint name="hokuyo_joint" type="continuous">
-    <origin xyz="-0.0446 0 0.0880" rpy="0 0 0" />
-    <parent link="head" />
-    <child link="hokuyo_link" />
-    <axis xyz="1 0 0" />
-    <dynamics damping="0.01" friction="0"/>
-  </joint>
-  <!-- Hokuyo Laser -->
-  <joint name="head_hokuyo_joint" type="fixed">
-    <axis xyz="0 1 0" />
-    <origin xyz="0.03 0 0.015" rpy="0 0 0"/>
-    <parent link="hokuyo_link"/>
-    <child link="head_hokuyo_frame"/>
-  </joint>
-  <link name="head_hokuyo_frame">
-    <inertial>
-      <mass value="1e-5" />
-      <!-- collocate with parent link and remove mass from it -->
-      <origin xyz="0.042428 0.0004084 0.0108165" rpy="0 0 0"/>
-      <inertia ixx="1e-6" ixy="0" ixz="0" iyy="1e-6" iyz="0" izz="1e-6" />
-    </inertial>
-  </link>
-  <link name="hokuyo_link">
-    <inertial>
-      <origin xyz="0.032428 0.0004084 -0.0041835" rpy="0 0 0" />
-      <mass value="0.057654" />
+  <joint name="${prefix}/left_camera_optical_joint" type="continuous">
+    <parent link="${prefix}/left_camera_optical_frame" />
+    <child link="${prefix}/motor" />
+  </joint>
+  <link name="${prefix}/motor"/>
+  <link name="${prefix}/spindle"/>
+  <joint name="${prefix}/motor_joint" type="continuous">
+    <parent link="${prefix}/motor" />
+    <child link="${prefix}/spindle" />
+    <axis xyz="0 0 1" />
+  </joint>
+  <joint name="{prefix}/spindle_joint" type="continuous">
+    <parent link="${prefix}/spindle" />
+    <child link="${prefix}/hokuyo_link" />
+  </joint>
+  <link name="${prefix}/hokuyo_link">
+    <inertial>
+      <origin xyz="0.012428 0.0004084 -0.0041835" rpy="0 0 0" />
+      <mass value="0.057664" />
       <inertia iyy="4.2412E-05" ixy="4.9927E-08" iyz="-9.8165E-09" ixx="3.7174E-05" ixz="1.1015E-05" izz="4.167E-05" />
     </inertial>
     <visual>
-      <!--origin xyz="0.065774 -0.001163 -0.08809" rpy="0 0 0" /-->
-      <!--origin xyz="0.045 -0.001163 -0.08809" rpy="-0.314 0 0" /-->
-      <origin xyz="0.045 -0.0261018277 -0.08342369" rpy="-0.314 0 0" />
+      <origin xyz="-.03 -.1 0" rpy="-1.9179632679 -1.57079632679 0" />
       <geometry>
         <mesh filename="package://multisense_description/meshes/head_camera.dae" />
@@ -76,10 +66,4 @@
     </visual>
   <collision>
-    <origin xyz="0.01885 0 -0.02119" rpy="0 0 0" />
-    <geometry>
-      <box size="0.08 0.06 0.04238"/>
-    </geometry>
-  </collision>
-  <collision>
     <origin xyz="0.03 0 0.0235" rpy="0 0 0" />
     <geometry>
@@ -88,12 +72,24 @@
   </collision>
   </link>
+  <link name="${prefix}/head_hokuyo_frame"/>
+  <joint name="${prefix}/head_hokuyo_frame_joint" type="fixed">
+    <!--
+     This transform accounts for the fact ROS expects laser data in the x forward,
+     y left, z up frame and the calibraton has the data in x left, y up, z forward.
+     Thus a roll of -90 * a pitch of -90 will make the appropriate transform. Note
+     Roll and pitch are both with respect to the origional x left, y up, z forward frame
+     -->
+    <origin xyz="0 0 0" rpy="-1.57079632679 -1.57079632679 0.0" />
+    <parent link="${prefix}/hokuyo_link" />
+    <child link="${prefix}/head_hokuyo_frame"/>
+  </joint>
   <!-- Stereo Camera -->
-  <joint name="left_camera_frame_joint" type="fixed">
+  <joint name="{prefix}/left_camera_frame_joint" type="fixed">
     <!-- optical frame collocated with tilting DOF -->
     <origin xyz="0.0 0.035 -0.002"/>
     <parent link="head"/>
-    <child link="left_camera_frame"/>
-  </joint>
-  <link name="left_camera_frame">
+    <child link="${prefix}/left_camera_frame"/>
+  </joint>
+  <link name="${prefix}/left_camera_frame">
     <inertial>
       <mass value="0.1" />
@@ -102,16 +98,16 @@
     </inertial>
   </link>
-  <joint name="left_camera_optical_frame_joint" type="fixed">
+  <joint name="{prefix}/left_camera_optical_frame_joint" type="fixed">
     <origin xyz="0 0 0" rpy="-1.57079632679 0.0 -1.57079632679" />
-    <parent link="left_camera_frame" />
-    <child link="left_camera_optical_frame"/>
-  </joint>
-  <link name="left_camera_optical_frame"/>
-  <joint name="right_camera_frame_joint" type="fixed">
+    <parent link="${prefix}/left_camera_frame" />
+    <child link="${prefix}/left_camera_optical_frame"/>
+  </joint>
+  <link name="${prefix}/left_camera_optical_frame"/>
+  <joint name="${prefix}/right_camera_frame_joint" type="fixed">
     <origin xyz="0.0 -0.035 -0.002"/>
     <parent link="head"/>
-    <child link="right_camera_frame"/>
-  </joint>
-  <link name="right_camera_frame">
+    <child link="${prefix}/right_camera_frame"/>
+  </joint>
+  <link name="${prefix}/right_camera_frame">
     <inertial>
       <mass value="0.1" />
@@ -120,52 +116,52 @@
     </inertial>
   </link>
-  <joint name="right_camera_optical_frame_joint" type="fixed">
+  <joint name="${prefix}/right_camera_optical_frame_joint" type="fixed">
     <origin xyz="0 0 0" rpy="-1.5708 0.0 -1.5708" />
-    <parent link="right_camera_frame" />
-    <child link="right_camera_optical_frame"/>
-  </joint>
-  <link name="right_camera_optical_frame"/>
-  <joint name="center_top_led_frame_joint" type="fixed">
+    <parent link="${prefix}/right_camera_frame" />
+    <child link="${prefix}/right_camera_optical_frame"/>
+  </joint>
+  <link name="${prefix}/right_camera_optical_frame"/>
+  <joint name="${prefix}/center_top_led_frame_joint" type="fixed">
     <origin xyz="0.01125 0.0 0.0105"/>
     <parent link="head"/>
-    <child link="center_top_led_frame"/>
-  </joint>
-  <link name="center_top_led_frame">
-    <inertial>
-      <mass value="0.1"/>
-      <origin xyz="0 0 0"/>
-      <inertia ixx="0.001" ixy="0.0" ixz="0.0" iyy="0.001" iyz="0.0" izz="0.001"/>
-    </inertial>
-  </link>
-  <joint name="center_bottom_led_frame_joint" type="fixed">
+    <child link="${prefix}/center_top_led_frame"/>
+  </joint>
+  <link name="${prefix}/center_top_led_frame">
+    <inertial>
+      <mass value="0.1"/>
+      <origin xyz="0 0 0"/>
+      <inertia ixx="0.001" ixy="0.0" ixz="0.0" iyy="0.001" iyz="0.0" izz="0.001"/>
+    </inertial>
+  </link>
+  <joint name="${prefix}/center_bottom_led_frame_joint" type="fixed">
     <origin xyz="0.01125 0.0 -0.0155"/>
     <parent link="head"/>
-    <child link="center_bottom_led_frame"/>
-  </joint>
-  <link name="center_bottom_led_frame">
-    <inertial>
-      <mass value="0.1"/>
-      <origin xyz="0 0 0"/>
-      <inertia ixx="0.001" ixy="0.0" ixz="0.0" iyy="0.001" iyz="0.0" izz="0.001"/>
-    </inertial>
-  </link>
-  <joint name="left_led_frame_joint" type="fixed">
+    <child link="${prefix}/center_bottom_led_frame"/>
+  </joint>
+  <link name="${prefix}/center_bottom_led_frame">
+    <inertial>
+      <mass value="0.1"/>
+      <origin xyz="0 0 0"/>
+      <inertia ixx="0.001" ixy="0.0" ixz="0.0" iyy="0.001" iyz="0.0" izz="0.001"/>
+    </inertial>
+  </link>
+  <joint name="${prefix}/left_led_frame_joint" type="fixed">
     <origin xyz="-0.01443 0.07452 0.050346" rpy="0 -0.15 0.53"/>
     <parent link="head"/>
-    <child link="left_led_frame"/>
-  </joint>
-  <link name="left_led_frame">
-    <inertial>
-      <mass value="0.1"/>
-      <origin xyz="0 0 0"/>
-      <inertia ixx="0.001" ixy="0.0" ixz="0.0" iyy="0.001" iyz="0.0" izz="0.001"/>
-    </inertial>
-  </link>
-  <joint name="right_led_frame_joint" type="fixed">
+    <child link="${prefix}/left_led_frame"/>
+  </joint>
+  <link name="${prefix}/left_led_frame">
+    <inertial>
+      <mass value="0.1"/>
+      <origin xyz="0 0 0"/>
+      <inertia ixx="0.001" ixy="0.0" ixz="0.0" iyy="0.001" iyz="0.0" izz="0.001"/>
+    </inertial>
+  </link>
+  <joint name="{prefix}/right_led_frame_joint" type="fixed">
     <origin xyz="-0.01443 -0.07452 0.050346" rpy="0 -0.15 -0.53"/>
     <parent link="head"/>
-    <child link="right_led_frame"/>
-  </joint>
-  <link name="right_led_frame">
+    <child link="${prefix}/right_led_frame"/>
+  </joint>
+  <link name="${prefix}/right_led_frame">
     <inertial>
       <mass value="0.1"/>
@@ -177,5 +173,5 @@
   <!-- Include transfrom to the left_camera_frame (shift in -.035mm in X and -.002mm in Z) -->
   <!-- imu link -->
-  <link name="head_imu_link">
+  <link name="${prefix}/head_imu_link">
     <inertial>
       <mass value="1e-5" />
@@ -191,29 +187,28 @@
     </visual>
   </link>
-  <joint name="head_imu_joint" type="fixed">
-    <parent link="head"/>
-    <child link="head_imu_link"/>
+  <joint name="${prefix}/head_imu_joint" type="fixed">
+    <parent link="head"/>
+    <child link="${prefix}/head_imu_link"/>
     <!-- putting it at the same z-level as the stereo -->
     <origin xyz="-0.0475 0.035 0.0" rpy="0 0 0"/>
   </joint>
   <xacro:multisense_sl_sensor prefix="hyq"/>
-      <!-- IMU definition -->
-  <link name="accel"/>
-  <joint name="accel_joint" type="fixed">
+  <link name="${prefix}/accel"/>
+  <joint name="${prefix}/accel_joint" type="fixed">
     <origin xyz="-.0475 .0302 -.00275" rpy="0 1.5707 0"/>
     <parent link="head_root"/>
-    <child link="accel"/>
-  </joint>
-  <link name="mag"/>
-  <joint name="mag_joint" type="fixed">
+    <child link="${prefix}/accel"/>
+  </joint>
+  <link name="${prefix}/mag"/>
+  <joint name="${prefix}/mag_joint" type="fixed">
     <origin xyz="-.0475 .0302 -.00275" rpy="0 1.5707 0"/>
     <parent link="head_root"/>
-    <child link="mag"/>
-  </joint>
-  <link name="gyro"/>
-  <joint name="gyro_joint" type="fixed">
+    <child link="${prefix}/mag"/>
+  </joint>
+  <link name="${prefix}/gyro"/>
+  <joint name="${prefix}/gyro_joint" type="fixed">
     <origin xyz="-.0476 .0388 -.00075" rpy="1.5707 3.14159 1.5707 "/>
     <parent link="head_root"/>
-    <child link="gyro"/>
+    <child link="${prefix}/gyro"/>
   </joint>
 </xacro:macro>

Commit message: [cleanup] Removed useless description of transmission for the hokuyo link
Note that these transmission are use for ros_control, and we're not
controlling this joint used ros_control. The joint control comes from
the  sensor driver (in simulation the sensors plugin).

File: urdfs/sensors/multisense_sl.gazebo.xacro (robot description, xacro)
@@ -173,14 +173,4 @@
 			<plugin filename="libMultiSenseSLPlugin.so" name="multisense_plugin"/>
 		</gazebo>
-		<transmission name="${prefix}/hokuyo_trans">
-			<type>transmission_interface/SimpleTransmission</type>
-			<joint name="${prefix}/hokuyo_joint">
-				<hardwareInterface>EffortJointInterface</hardwareInterface>
-			</joint>
-			<actuator name="${prefix}/hokuyo_motor">
-				<hardwareInterface>EffortJointInterface</hardwareInterface>
-				<mechanicalReduction>1</mechanicalReduction>
-			</actuator>
-		</transmission>
 	</xacro:macro>
 </robot>

Commit message: [feature] This modifications should be compatible with simulation and real sensor driver

File: urdfs/sensors/multisense_sl.gazebo.xacro (robot description, xacro)
@@ -18,5 +18,5 @@
 			<mu2>0.9</mu2>
 		</gazebo>
-		<gazebo reference="${prefix}/head_hokuyo_frame_joint">
+		<gazebo reference="${prefix}/motor_joint">
 			<implicitSpringDamper>1</implicitSpringDamper>
 		</gazebo>

File: urdfs/sensors/multisense_sl.urdf.xacro (robot description, xacro)
@@ -1,4 +1,5 @@
 <?xml version="1.0" ?>
 <robot xmlns:xacro="http://ros.org/wiki/xacro">
+<xacro:include filename="$(find sensors_description)/urdfs/sensors/multisense_sl.gazebo.xacro"/>
 <xacro:macro name="multisense_sl" params="parent *origin prefix" >
 	<joint name="${parent}_head_root_joint" type="fixed">
@@ -8,12 +9,19 @@
 	</joint>
 	<!-- Multisense joints -->
-	<link name="head_root"/>
+	<link name="head_root">
+		<inertial>
+			<mass value="0.001" />
+			<origin xyz="0 0 0" />
+			<inertia ixx="0.001"  ixy="0.0"  ixz="0.0" iyy="0.001"  iyz="0.0" izz="0.001" />
+		</inertial>
+	</link>
 	<joint name="head_root_joint" type="fixed">
 		<parent link="head_root"/>
 		<child link="head"/>
 	</joint>
-	<joint name="${prefix}/left_camera_optical_joint" type="continuous">
+	<joint name="${prefix}/left_camera_optical_joint" type="fixed">
 		<parent link="${prefix}/left_camera_optical_frame" />
 		<child link="${prefix}/motor" />
+		<origin xyz="0.027 -0.097 -0.017" rpy="0. 0. 2." />
 	</joint>
 	<joint name="${prefix}/motor_joint" type="continuous">
@@ -22,7 +30,8 @@
 		<axis xyz="0 0 1" />
 	</joint>
-	<joint name="{prefix}/spindle_joint" type="continuous">
+	<joint name="${prefix}/spindle_joint" type="fixed">
 		<parent link="${prefix}/spindle" />
 		<child link="${prefix}/hokuyo_link" />
+		<origin xyz="0.001 0.01 0.0" rpy="0. 0. 0." />
 	</joint>
 	<joint name="${prefix}/head_hokuyo_frame_joint" type="fixed">
@@ -38,5 +47,5 @@
 	</joint>
 	<!-- Stereo Camera -->
-	<joint name="{prefix}/left_camera_frame_joint" type="fixed">
+	<joint name="${prefix}/left_camera_frame_joint" type="fixed">
 		<!-- optical frame collocated with tilting DOF -->
 		<origin xyz="0.0 0.035 -0.002"/>
@@ -44,5 +53,5 @@
 		<child link="${prefix}/left_camera_frame"/>
 	</joint>
-	<joint name="{prefix}/left_camera_optical_frame_joint" type="fixed">
+	<joint name="${prefix}/left_camera_optical_frame_joint" type="fixed">
 		<origin xyz="0 0 0" rpy="-1.57079632679 0.0 -1.57079632679" />
 		<parent link="${prefix}/left_camera_frame" />
@@ -74,5 +83,5 @@
 		<child link="${prefix}/left_led_frame"/>
 	</joint>
-	<joint name="{prefix}/right_led_frame_joint" type="fixed">
+	<joint name="${prefix}/right_led_frame_joint" type="fixed">
 		<origin xyz="-0.01443 -0.07452 0.050346" rpy="0 -0.15 -0.53"/>
 		<parent link="head"/>
@@ -123,6 +132,18 @@
 		</collision>
 	</link>
-	<link name="${prefix}/motor"/>
-	<link name="${prefix}/spindle"/>
+	<link name="${prefix}/motor">
+		<inertial>
+			<mass value="0.001" />
+			<origin xyz="0 0 0" />
+			<inertia ixx="0.001"  ixy="0.0"  ixz="0.0" iyy="0.001"  iyz="0.0" izz="0.001" />
+		</inertial>
+	</link>
+	<link name="${prefix}/spindle">
+		<inertial>
+			<mass value="0.001" />
+			<origin xyz="0 0 0" />
+			<inertia ixx="0.001"  ixy="0.0"  ixz="0.0" iyy="0.001"  iyz="0.0" izz="0.001" />
+		</inertial>
+	</link>
 	<link name="${prefix}/hokuyo_link">
 		<inertial>
@@ -147,5 +168,11 @@
 		</collision>
 	</link>
-	<link name="${prefix}/head_hokuyo_frame"/>
+	<link name="${prefix}/head_hokuyo_frame">
+		<inertial>
+			<mass value="0.001" />
+			<origin xyz="0 0 0" />
+			<inertia ixx="0.001"  ixy="0.0"  ixz="0.0" iyy="0.001"  iyz="0.0" izz="0.001" />
+		</inertial>
+	</link>
 	<link name="${prefix}/left_camera_frame">
 		<inertial>
@@ -155,5 +182,11 @@
 		</inertial>
 	</link>
-	<link name="${prefix}/left_camera_optical_frame"/>
+	<link name="${prefix}/left_camera_optical_frame">
+		<inertial>
+			<mass value="0.001" />
+			<origin xyz="0 0 0" />
+			<inertia ixx="0.001"  ixy="0.0"  ixz="0.0" iyy="0.001"  iyz="0.0" izz="0.001" />
+		</inertial>
+	</link>
 	<link name="${prefix}/right_camera_frame">
 		<inertial>
@@ -163,5 +196,11 @@
 		</inertial>
 	</link>
-	<link name="${prefix}/right_camera_optical_frame"/>
+	<link name="${prefix}/right_camera_optical_frame">
+		<inertial>
+			<mass value="0.001" />
+			<origin xyz="0 0 0" />
+			<inertia ixx="0.001"  ixy="0.0"  ixz="0.0" iyy="0.001"  iyz="0.0" izz="0.001" />
+		</inertial>
+	</link>
 	<link name="${prefix}/center_top_led_frame">
 		<inertial>
@@ -213,5 +252,5 @@
 	<link name="${prefix}/gyro"/>
 	<!-- Gazebo multisense plugin -->
-	<xacro:multisense_sl_sensor prefix="hyq"/>
+	<xacro:multisense_sl_sensor prefix="${prefix}"/>
 </xacro:macro>
 </robot>

Commit message: adding robot name as parameter
WARNING: removed extra rotation to compensate Multisense Hokuyo
It might not work on real robot!!!

File: urdfs/sensors/multisense_sl.gazebo.xacro (robot description, xacro)
@@ -1,5 +1,5 @@
 <?xml version="1.0"?>
 <robot xmlns:xacro="http://ros.org/wiki/xacro">
-	<xacro:macro name="multisense_sl_sensor" params="prefix">
+	<xacro:macro name="multisense_sl_sensor" params="prefix robot_name">
 		<gazebo reference="head_root">
 			<mu1>0.9</mu1>
@@ -66,5 +66,5 @@
 				<image>
 					<width>1024</width>
-					<height>544</height>
+                    <height>1024</height>
 					<format>R8G8B8</format>
 				</image>
@@ -92,5 +92,5 @@
 				<image>
 					<width>1024</width>
-					<height>544</height>
+                    <height>1024</height>
 					<format>R8G8B8</format>
 				</image>
@@ -114,9 +114,9 @@
 				<alwaysOn>true</alwaysOn>
 				<updateRate>0.0</updateRate>
-				<cameraName>${prefix}/camera</cameraName>
-				<imageTopicName>image_color</imageTopicName>
-				<cameraInfoTopicName>camera_info</cameraInfoTopicName>
-				<frameName>${prefix}/left_camera_optical_frame</frameName>
-				<!--<rightFrameName>right_camera_optical_frame</rightFrameName>-->
+                <cameraName>${prefix}/camera</cameraName>
+                <imageTopicName>image_color</imageTopicName>
+                <cameraInfoTopicName>camera_info</cameraInfoTopicName>
+                <frameName>${prefix}/left_camera_optical_frame</frameName>
+                <rightFrameName>${prefix}/right_camera_optical_frame</rightFrameName>
 				<hackBaseline>0.07</hackBaseline>
 				<distortionK1>0.0</distortionK1>
@@ -171,6 +171,8 @@
 		</gazebo>
 		<gazebo>
-			<plugin filename="libMultiSenseSLPlugin.so" name="multisense_plugin"/>
+			<plugin filename="libMultiSenseSLPlugin.so" name="multisense_plugin">
+                <robot_name>${robot_name}</robot_name>
+            </plugin>
 		</gazebo>
-	</xacro:macro>
+     </xacro:macro>
 </robot>

File: urdfs/sensors/multisense_sl.urdf.xacro (robot description, xacro)
@@ -2,5 +2,5 @@
 <robot xmlns:xacro="http://ros.org/wiki/xacro">
 <xacro:include filename="$(find sensors_description)/urdfs/sensors/multisense_sl.gazebo.xacro"/>
-<xacro:macro name="multisense_sl" params="parent *origin prefix" >
+<xacro:macro name="multisense_sl" params="parent *origin prefix robot_name" >
 	<joint name="${parent}_head_root_joint" type="fixed">
 		<insert_block name="origin"/>
@@ -42,5 +42,6 @@
 		Roll and pitch are both with respect to the origional x left, y up, z forward frame
 		-->
-		<origin xyz="0 0 0" rpy="-1.57079632679 -1.57079632679 0.0" />
+		<!--origin xyz="0 0 0" rpy="-1.57079632679 -1.57079632679 0.0" /-->
+                <origin xyz="0 0 0" rpy="0 0 0" />
 		<parent link="${prefix}/hokuyo_link" />
 		<child link="${prefix}/head_hokuyo_frame"/>
@@ -252,5 +253,5 @@
 	<link name="${prefix}/gyro"/>
 	<!-- Gazebo multisense plugin -->
-	<xacro:multisense_sl_sensor prefix="${prefix}"/>
+	<xacro:multisense_sl_sensor prefix="${prefix}" robot_name="${robot_name}"/>
 </xacro:macro>
 </robot>
