Commit message: Revert "adding robot name as parameter"
This reverts commit a4868601ba7b09185282c47406d83819b4dea729.

Conflicts:
	urdfs/sensors/multisense_sl.gazebo.xacro

File: urdfs/sensors/multisense_sl.gazebo.xacro (robot description, xacro)
@@ -1,5 +1,5 @@
 <?xml version="1.0"?>
 <robot xmlns:xacro="http://ros.org/wiki/xacro">
-	<xacro:macro name="multisense_sl_sensor" params="prefix robot_name">
+	<xacro:macro name="multisense_sl_sensor" params="prefix">
 		<gazebo reference="head_root">
 			<mu1>0.9</mu1>
@@ -176,7 +176,5 @@
 		</gazebo>
 		<gazebo>
-			<plugin filename="libMultiSenseSLPlugin.so" name="multisense_plugin">
-                <robot_name>${robot_name}</robot_name>
-            </plugin>
+			<plugin filename="libMultiSenseSLPlugin.so" name="multisense_plugin"/>
 		</gazebo>
      </xacro:macro>

File: urdfs/sensors/multisense_sl.urdf.xacro (robot description, xacro)
@@ -2,5 +2,5 @@
 <robot xmlns:xacro="http://ros.org/wiki/xacro">
 <xacro:include filename="$(find sensors_description)/urdfs/sensors/multisense_sl.gazebo.xacro"/>
-<xacro:macro name="multisense_sl" params="parent *origin prefix robot_name" >
+<xacro:macro name="multisense_sl" params="parent *origin prefix" >
 	<joint name="${parent}_head_root_joint" type="fixed">
 		<insert_block name="origin"/>
@@ -42,6 +42,5 @@
 		Roll and pitch are both with respect to the origional x left, y up, z forward frame
 		-->
-		<!--origin xyz="0 0 0" rpy="-1.57079632679 -1.57079632679 0.0" /-->
-                <origin xyz="0 0 0" rpy="0 0 0" />
+		<origin xyz="0 0 0" rpy="-1.57079632679 -1.57079632679 0.0" />
 		<parent link="${prefix}/hokuyo_link" />
 		<child link="${prefix}/head_hokuyo_frame"/>
@@ -253,5 +252,5 @@
 	<link name="${prefix}/gyro"/>
 	<!-- Gazebo multisense plugin -->
-	<xacro:multisense_sl_sensor prefix="${prefix}" robot_name="${robot_name}"/>
+	<xacro:multisense_sl_sensor prefix="${prefix}"/>
 </xacro:macro>
 </robot>

Commit message: Simulated static transforms are now the same as on the real sensor

File: urdfs/sensors/multisense_sl.gazebo.xacro (robot description, xacro)
@@ -19,4 +19,10 @@
 		</gazebo>
 		<gazebo reference="${prefix}/motor_joint">
+			<implicitSpringDamper>1</implicitSpringDamper>
+		</gazebo>
+		<gazebo reference="${prefix}/left_camera_optical_joint">
+			<implicitSpringDamper>1</implicitSpringDamper>
+		</gazebo>
+		<gazebo reference="${prefix}/spindle_joint">
 			<implicitSpringDamper>1</implicitSpringDamper>
 		</gazebo>

File: urdfs/sensors/multisense_sl.urdf.xacro (robot description, xacro)
@@ -23,4 +23,5 @@
 		<parent link="${prefix}/left_camera_optical_frame" />
 		<child link="${prefix}/motor" />
+                <origin xyz="0.027155533433 -0.0971753746271 -0.0172099247575" rpy="0.00196935 0.00780759 2.06496" />
 	</joint>
 	<joint name="${prefix}/motor_joint" type="continuous">
@@ -32,4 +33,5 @@
 		<parent link="${prefix}/spindle" />
 		<child link="${prefix}/hokuyo_link" />
+                <origin xyz="0.000662488571834 0.00996151566505 -7.18757200957e-6" rpy="-0.00223496 -0.0227575 -1.53777e-12" />
 	</joint>
 	<joint name="${prefix}/head_hokuyo_frame_joint" type="fixed">
