Commit message: Substituted hyq with sensors for finding the files

File: urdfs/sensors/asus_xtion.urdf.xacro (robot description, xacro)
@@ -1,5 +1,5 @@
 <?xml version="1.0"?>
 <root xmlns:xacro="http://www.ros.org/wiki/xacro">
-	<xacro:include filename="$(find hyq_description)/urdfs/sensors/asus_xtion.gazebo.xacro" />
+	<xacro:include filename="$(find sensors_description)/urdfs/sensors/asus_xtion.gazebo.xacro" />
 	<!-- ===================================== ASUS & PROSILICA ==================================== -->
 	<!-- The xacro macro xacro:asus_xtion_camera contains: asus xtion and prosilica combo -->
@@ -46,5 +46,5 @@
 				<origin xyz="0 0 0" rpy="0 0 0"/>
 				<geometry>
-					<mesh filename="package://hyq_description/meshes/sensors/asus_xtion.dae" scale="1 1 1" />
+					<mesh filename="package://sensors_description/meshes/sensors/asus_xtion.dae" scale="1 1 1" />
 				</geometry>
 				<material name="gray">

File: urdfs/sensors/bumblebee.urdf.xacro (robot description, xacro)
@@ -1,5 +1,5 @@
 <?xml version="1.0"?>
 <robot xmlns:xacro="http://www.ros.org/wiki/xacro">
-	<xacro:include filename="$(find hyq_description)/urdfs/sensors/stereo_camera.gazebo.xacro"/>
+	<xacro:include filename="$(find sensors_description)/urdfs/sensors/stereo_camera.gazebo.xacro"/>
 	<!-- ================================ Bumblebee ============================== -->
 	<!-- The xacro macro xacro:bumblebee contains: camera, mount and optical frame -->
@@ -19,5 +19,5 @@
 				<origin xyz="0 0 0.018" rpy="${PI/2} 0 ${PI/2}"/>
 				<geometry>
-					<mesh filename="package://hyq_description/meshes/sensors/bumblebee.dae"/>
+					<mesh filename="package://sensors_description/meshes/sensors/bumblebee.dae"/>
 				</geometry>
 			</visual>
@@ -25,5 +25,5 @@
 				<origin xyz="0 0 0.018" rpy="${PI/2} 0 ${PI/2}"/>
 				<geometry>
-					<mesh filename="package://hyq_description/meshes/sensors/bumblebee.dae"/>
+					<mesh filename="package://sensors_description/meshes/sensors/bumblebee.dae"/>
 				</geometry>
 			</collision>

File: urdfs/sensors/hokuyo_laser.urdf.xacro (robot description, xacro)
@@ -23,5 +23,5 @@
 				<origin xyz="0 0 0" rpy="0 0 0" />
 				<geometry>
-					<mesh filename="package://hyq_description/meshes/sensors/hokuyo.dae" scale="0.0254 0.0254 0.0254" />
+					<mesh filename="package://sensors_description/meshes/sensors/hokuyo.dae" scale="0.0254 0.0254 0.0254" />
 				</geometry>
 			</visual>

File: urdfs/sensors/kinect.urdf.xacro (robot description, xacro)
@@ -1,5 +1,5 @@
 <?xml version="1.0"?>
 <root xmlns:xacro="http://www.ros.org/wiki/xacro">
-	<xacro:include filename="$(find hyq_description)/urdfs/sensors/kinect.gazebo.xacro" />
+	<xacro:include filename="$(find sensors_description)/urdfs/sensors/kinect.gazebo.xacro" />
 	<property name="ir_depth_rgb_offset_y" value="0.01"/> <!-- FIXME: what is this offset? -->
 	<!-- ===================================== KINECT & PROSILICA ==================================== -->
@@ -46,5 +46,5 @@
 				<origin xyz="0.0 0.0 0.0" rpy="0.0 0.0 0"/>
 				<geometry>
-					<mesh filename="package://hyq_description/meshes/sensors/kinect.dae" scale="1 1 1" />
+					<mesh filename="package://sensors_description/meshes/sensors/kinect.dae" scale="1 1 1" />
 				</geometry>
 				<material name="gray">
@@ -55,5 +55,5 @@
 				<origin xyz="0.0 0.0 0.0" rpy="0.0 0.0 0.0"/>
 				<geometry>
-					<mesh filename="package://hyq_description/meshes/sensors/kinect.dae" scale="1 1 1" />
+					<mesh filename="package://sensors_description/meshes/sensors/kinect.dae" scale="1 1 1" />
 				</geometry>
 			</collision>

File: urdfs/sensors/microstrain_3dmgx325_imu.urdf.xacro (robot description, xacro)
@@ -1,5 +1,5 @@
 <?xml version="1.0"?>
 <robot xmlns:xacro="http://ros.org/wiki/xacro">
-	<xacro:include filename="$(find hyq_description)/urdfs/sensors/microstrain_3dmgx325_imu.gazebo.xacro"/>
+	<xacro:include filename="$(find sensors_description)/urdfs/sensors/microstrain_3dmgx325_imu.gazebo.xacro"/>
 	<!-- ============================ IMU microstrain ============================== -->
 	<!-- The xacro macro xacro:microstrain_3dmgx325_imu: imu frame -->

File: urdfs/sensors/microstrain_3dmgx425_imu.urdf.xacro (robot description, xacro)
@@ -1,5 +1,5 @@
 <?xml version="1.0"?>
 <robot xmlns:xacro="http://ros.org/wiki/xacro">
-	<xacro:include filename="$(find hyq_description)/urdfs/sensors/microstrain_3dmgx425_imu.gazebo.xacro"/>
+	<xacro:include filename="$(find sensors_description)/urdfs/sensors/microstrain_3dmgx425_imu.gazebo.xacro"/>
 	<!-- ============================ IMU microstrain ============================== -->
 	<!-- The xacro macro xacro:microstrain_3dmgx425_imu: imu frame -->

File: urdfs/sensors/ptu_d46.urdf.xacro (robot description, xacro)
@@ -2,5 +2,5 @@
 <robot xmlns:xacro="http://www.ros.org/wiki/xacro">
 	<!-- Things that are needed only for Gazebo (not the physical robot). These include sensor and controller plugin specifications -->
-	<xacro:include filename="$(find hyq_description)/urdfs/sensors/ptu_d46.transmission.xacro"/>
+	<xacro:include filename="$(find sensors_description)/urdfs/sensors/ptu_d46.transmission.xacro"/>
 	<xacro:macro name="d46_stepper_module" params="ptu_name joint_name">
 		<link name="${ptu_name}_${joint_name}_link">

File: urdfs/sensors/velodyne.urdf.xacro (robot description, xacro)
@@ -1,5 +1,5 @@
 <?xml version="1.0"?>
 <robot xmlns:xacro="http://www.ros.org/wiki/xacro">
-	<xacro:include filename="$(find hyq_description)/urdfs/sensors/velodyne.gazebo.xacro" />
+	<xacro:include filename="$(find sensors_description)/urdfs/sensors/velodyne.gazebo.xacro" />
 	<!-- ===================================== VELODYNE ==================================== -->
 	<!-- The xacro macro xacro:velodyne contains: velodyne combo -->
@@ -27,5 +27,5 @@
 				<origin xyz="0 0 0" rpy="0 0 0"/>
 				<geometry>
-					<mesh filename="package://hyq_description/meshes/sensors/velodyne_hdl32e.dae" scale="1 1 1" />
+					<mesh filename="package://sensors_description/meshes/sensors/velodyne_hdl32e.dae" scale="1 1 1" />
 				</geometry>
 				<material name="gray">
@@ -36,5 +36,5 @@
 				<origin xyz="0 0 0" rpy="0 0 0"/>
 				<geometry>
-					<mesh filename="package://hyq_description/meshes/sensors/velodyne_hdl32e.dae" scale="1 1 1" />
+					<mesh filename="package://sensors_description/meshes/sensors/velodyne_hdl32e.dae" scale="1 1 1" />
 				</geometry>
 			</collision>

File: urdfs/sensors/vislab_3dve.urdf.xacro (robot description, xacro)
@@ -1,5 +1,5 @@
 <?xml version="1.0"?>
 <robot xmlns:xacro="http://www.ros.org/wiki/xacro">
-	<xacro:include filename="$(find hyq_description)/urdfs/sensors/stereo_camera.gazebo.xacro"/>
+	<xacro:include filename="$(find sensors_description)/urdfs/sensors/stereo_camera.gazebo.xacro"/>
 	<xacro:macro name="vislab_3dve" params="name parent xyz rpy high_res hfov">
 		<joint name="${name}_vislab_3dve_mount_joint" type="fixed">
@@ -18,5 +18,5 @@
 				<origin xyz="0.018 0 0" rpy="${PI/2} 0 ${-PI/2}"/>
 				<geometry>
-					<mesh filename="package://hyq_description/meshes/sensors/vislab_3dve.stl"/>
+					<mesh filename="package://sensors_description/meshes/sensors/vislab_3dve.stl"/>
 				</geometry>
 			</visual>
@@ -24,5 +24,5 @@
 				<origin xyz="0.018 0 0" rpy="${PI/2} 0 ${-PI/2}"/>
 				<geometry>
-					<mesh filename="package://hyq_description/meshes/sensors/vislab_3dve.stl"/>
+					<mesh filename="package://sensors_description/meshes/sensors/vislab_3dve.stl"/>
 				</geometry>
 			</collision>

Commit message: [config] Removing the inertia values of the sensors
The actual identification procedure doesn't consider the sensors masses
to compute the trunk mass. It produces differences between when you put
that value as trunk mass.

File: urdfs/sensors/asus_xtion.urdf.xacro (robot description, xacro)
@@ -39,5 +39,5 @@
 		<link name="${name}_mount_link">
 			<inertial>
-				<mass value="0.1"/>
+				<mass value="0.001"/>
 				<origin xyz="0 0 0" rpy="0 0 0"/>
 				<inertia ixx="0.01" ixy="0.0" ixz="0.0" iyy="0.01" iyz="0.0" izz="0.01"/>
@@ -62,5 +62,5 @@
 		<link name="${name}_depth_frame">
 			<inertial>
-				<mass value="0.1" />
+				<mass value="0.001" />
 				<origin xyz="0 0 0" rpy="0 0 0"/>
 				<inertia ixx="0.01" ixy="0.0" ixz="0.0" iyy="0.01" iyz="0.0" izz="0.01"/>
@@ -84,5 +84,5 @@
 		<link name="${name}_rgb_frame" >
 			<inertial>
-				<mass value="0.1" />
+				<mass value="0.001" />
 				<origin xyz="0 0 0" rpy="0 0 0"/>
 				<inertia ixx="0.01" ixy="0.0" ixz="0.0" iyy="0.01" iyz="0.0" izz="0.01" />

File: urdfs/sensors/multisense_sl.urdf.xacro (robot description, xacro)
@@ -111,5 +111,6 @@
 		<inertial>
 			<origin xyz="-0.075493 3.3383E-05 0.02774" rpy="0 0 0" />
-			<mass value="1.4199" />
+			<!--<mass value="1.4199" />-->
+			<mass value="0.001" />
 			<inertia iyy="0.0041178" ixy="-1.5797E-06" iyz="-6.8415E-07" ixx="0.0039688" ixz="-0.00089293" izz="0.0035243" />
 		</inertial>
@@ -147,5 +148,5 @@
 		<inertial>
 			<origin xyz="0.012428 0.0004084 -0.0041835" rpy="0 0 0" />
-			<mass value="0.057664" />
+			<mass value="0.001" />
 			<inertia iyy="4.2412E-05" ixy="4.9927E-08" iyz="-9.8165E-09" ixx="3.7174E-05" ixz="1.1015E-05" izz="4.167E-05" />
 		</inertial>
@@ -175,5 +176,5 @@
 	<link name="${prefix}/left_camera_frame">
 		<inertial>
-			<mass value="0.1" />
+			<mass value="0.001" />
 			<origin xyz="0 0 0" />
 			<inertia ixx="0.001"  ixy="0.0"  ixz="0.0" iyy="0.001"  iyz="0.0" izz="0.001" />
@@ -189,5 +190,5 @@
 	<link name="${prefix}/right_camera_frame">
 		<inertial>
-			<mass value="0.1" />
+			<mass value="0.001" />
 			<origin xyz="0 0 0" />
 			<inertia ixx="0.001"  ixy="0.0"  ixz="0.0" iyy="0.001"  iyz="0.0" izz="0.001" />
@@ -203,5 +204,5 @@
 	<link name="${prefix}/center_top_led_frame">
 		<inertial>
-			<mass value="0.1"/>
+			<mass value="0.001"/>
 			<origin xyz="0 0 0"/>
 			<inertia ixx="0.001" ixy="0.0" ixz="0.0" iyy="0.001" iyz="0.0" izz="0.001"/>
@@ -210,5 +211,5 @@
 	<link name="${prefix}/center_bottom_led_frame">
 		<inertial>
-			<mass value="0.1"/>
+			<mass value="0.001"/>
 			<origin xyz="0 0 0"/>
 				<inertia ixx="0.001" ixy="0.0" ixz="0.0" iyy="0.001" iyz="0.0" izz="0.001"/>
@@ -217,5 +218,5 @@
 	<link name="${prefix}/left_led_frame">
 		<inertial>
-			<mass value="0.1"/>
+			<mass value="0.001"/>
 			<origin xyz="0 0 0"/>
 			<inertia ixx="0.001" ixy="0.0" ixz="0.0" iyy="0.001" iyz="0.0" izz="0.001"/>
@@ -224,5 +225,5 @@
 	<link name="${prefix}/right_led_frame">
 		<inertial>
-			<mass value="0.1"/>
+			<mass value="0.001"/>
 			<origin xyz="0 0 0"/>
 			<inertia ixx="0.001" ixy="0.0" ixz="0.0" iyy="0.001" iyz="0.0" izz="0.001"/>

Commit message: [config] Removing the inertia values of the sensors
The actual identification procedure doesn't consider the sensors masses
to compute the trunk mass. It produces differences between when you put
that value as trunk mass.

File: urdfs/sensors/asus_xtion.urdf.xacro (robot description, xacro)
@@ -39,5 +39,5 @@
 		<link name="${name}_mount_link">
 			<inertial>
-				<mass value="0.1"/>
+				<mass value="0.001"/>
 				<origin xyz="0 0 0" rpy="0 0 0"/>
 				<inertia ixx="0.01" ixy="0.0" ixz="0.0" iyy="0.01" iyz="0.0" izz="0.01"/>
@@ -62,5 +62,5 @@
 		<link name="${name}_depth_frame">
 			<inertial>
-				<mass value="0.1" />
+				<mass value="0.001" />
 				<origin xyz="0 0 0" rpy="0 0 0"/>
 				<inertia ixx="0.01" ixy="0.0" ixz="0.0" iyy="0.01" iyz="0.0" izz="0.01"/>
@@ -84,5 +84,5 @@
 		<link name="${name}_rgb_frame" >
 			<inertial>
-				<mass value="0.1" />
+				<mass value="0.001" />
 				<origin xyz="0 0 0" rpy="0 0 0"/>
 				<inertia ixx="0.01" ixy="0.0" ixz="0.0" iyy="0.01" iyz="0.0" izz="0.01" />

File: urdfs/sensors/multisense_sl.urdf.xacro (robot description, xacro)
@@ -113,5 +113,6 @@
 		<inertial>
 			<origin xyz="-0.075493 3.3383E-05 0.02774" rpy="0 0 0" />
-			<mass value="1.4199" />
+			<!--<mass value="1.4199" />-->
+			<mass value="0.001" />
 			<inertia iyy="0.0041178" ixy="-1.5797E-06" iyz="-6.8415E-07" ixx="0.0039688" ixz="-0.00089293" izz="0.0035243" />
 		</inertial>
@@ -149,5 +150,5 @@
 		<inertial>
 			<origin xyz="0.012428 0.0004084 -0.0041835" rpy="0 0 0" />
-			<mass value="0.057664" />
+			<mass value="0.001" />
 			<inertia iyy="4.2412E-05" ixy="4.9927E-08" iyz="-9.8165E-09" ixx="3.7174E-05" ixz="1.1015E-05" izz="4.167E-05" />
 		</inertial>
@@ -177,5 +178,5 @@
 	<link name="${prefix}/left_camera_frame">
 		<inertial>
-			<mass value="0.1" />
+			<mass value="0.001" />
 			<origin xyz="0 0 0" />
 			<inertia ixx="0.001"  ixy="0.0"  ixz="0.0" iyy="0.001"  iyz="0.0" izz="0.001" />
@@ -191,5 +192,5 @@
 	<link name="${prefix}/right_camera_frame">
 		<inertial>
-			<mass value="0.1" />
+			<mass value="0.001" />
 			<origin xyz="0 0 0" />
 			<inertia ixx="0.001"  ixy="0.0"  ixz="0.0" iyy="0.001"  iyz="0.0" izz="0.001" />
@@ -205,5 +206,5 @@
 	<link name="${prefix}/center_top_led_frame">
 		<inertial>
-			<mass value="0.1"/>
+			<mass value="0.001"/>
 			<origin xyz="0 0 0"/>
 			<inertia ixx="0.001" ixy="0.0" ixz="0.0" iyy="0.001" iyz="0.0" izz="0.001"/>
@@ -212,5 +213,5 @@
 	<link name="${prefix}/center_bottom_led_frame">
 		<inertial>
-			<mass value="0.1"/>
+			<mass value="0.001"/>
 			<origin xyz="0 0 0"/>
 				<inertia ixx="0.001" ixy="0.0" ixz="0.0" iyy="0.001" iyz="0.0" izz="0.001"/>
@@ -219,5 +220,5 @@
 	<link name="${prefix}/left_led_frame">
 		<inertial>
-			<mass value="0.1"/>
+			<mass value="0.001"/>
 			<origin xyz="0 0 0"/>
 			<inertia ixx="0.001" ixy="0.0" ixz="0.0" iyy="0.001" iyz="0.0" izz="0.001"/>
@@ -226,5 +227,5 @@
 	<link name="${prefix}/right_led_frame">
 		<inertial>
-			<mass value="0.1"/>
+			<mass value="0.001"/>
 			<origin xyz="0 0 0"/>
 			<inertia ixx="0.001" ixy="0.0" ixz="0.0" iyy="0.001" iyz="0.0" izz="0.001"/>
