Commit message: Extended FOV of sensors for FASTER stair climbing simulation

File: urdfs/sensors/asus_xtion.gazebo.xacro (robot description, xacro)
@@ -29,5 +29,5 @@
 					<pointCloudTopicName>/${camera_name}/depth/points</pointCloudTopicName>
 					<frameName>${frame_name}</frameName>
-					<pointCloudCutoff>0.5</pointCloudCutoff>
+					<pointCloudCutoff>0.05</pointCloudCutoff>
 					<distortionK1>0.00000001</distortionK1>
 					<distortionK2>0.00000001</distortionK2>
@@ -51,5 +51,5 @@
 				<update_rate>30.0</update_rate>
 				<camera>
-					<horizontal_fov>${58.0*PI/180.0}</horizontal_fov>
+					<horizontal_fov>${100.0*PI/180.0}</horizontal_fov>
 					<image>
 						<format>R8G8B8</format>
@@ -58,6 +58,6 @@
 					</image>
 					<clip>
-						<near>0.48</near>
-						<far>3.5</far>
+						<near>0.1</near>
+						<far>1</far>
 					</clip>
 				</camera>
@@ -72,5 +72,5 @@
 					<pointCloudTopicName>/${camera_name}/depth_registered/points</pointCloudTopicName>
 					<frameName>${frame_name}</frameName>
-					<pointCloudCutoff>0.5</pointCloudCutoff>
+					<pointCloudCutoff>0.01</pointCloudCutoff>
 					<distortionK1>0.00000001</distortionK1>
 					<distortionK2>0.00000001</distortionK2>

File: urdfs/sensors/asus_xtion.urdf.xacro (robot description, xacro)
@@ -52,10 +52,10 @@
 				</material>
 			</visual>
-			<collision>
+			<!--<collision>
 				<origin xyz="0 0 ${asus_xtion_z}" rpy="0 0 0" />
 				<geometry>
 					<box size="0.05 .18 0.035" />
 				</geometry>
-			</collision>
+			</collision>-->
 		</link>
 		<!-- ir sensor link -->
@@ -72,10 +72,10 @@
 				</geometry>
 			</visual>
-			<collision>
+			<!--<collision>
 				<origin xyz="0 0 0" rpy="0 0 0"/>
 				<geometry>
 					<sphere radius="0.0005"/>
 				</geometry>
-			</collision>
+			</collision>-->
 		</link>
 		<!-- ir optical sensor link -->
@@ -94,10 +94,10 @@
 				</geometry>
 			</visual>
-			<collision>
+			<!--<collision>
 				<origin xyz="0 0 0" rpy="0 0 0"/>
 				<geometry>
 					<sphere radius="0.0005"/>
 				</geometry>
-			</collision>
+			</collision>-->
 		</link>
 		<!-- rgb optical sensor link -->

File: urdfs/sensors/multisense_sl.urdf.xacro (robot description, xacro)
@@ -126,10 +126,10 @@
 			</material>
 		</visual>
-		<collision>
+	<!--	<collision>
 			<origin xyz="-0.0503 0 -0.00195" rpy="0 0 0" />
 			<geometry>
 				<box size="0.1311 0.12 0.0591"/>
 			</geometry>
-		</collision>
+		</collision>-->
 	</link>
 	<link name="${prefix}/motor">
@@ -162,10 +162,10 @@
 			</material>
 		</visual>
-		<collision>
+		<!--<collision>
 			<origin xyz="0.03 0 0.0235" rpy="0 0 0" />
 			<geometry>
 				<cylinder radius="0.024425" length="0.047"/>
 			</geometry>
-		</collision>
+		</collision>-->
 	</link>
 	<link name="${prefix}/head_hokuyo_frame">
