Commit message: [cleanup] Improving the spaces of the code lines

File: urdfs/sensors/kvh_1775_imu.urdf.xacro (robot description, xacro)
@@ -25,7 +25,7 @@
 					<cylinder radius="0.0482" length="0.0737" />
 				</geometry>
-                                <material name="aluminium">
-                                	<color rgba="0.35 0.35 0.35 1" />
-                                </material>
+					<material name="aluminium">
+						<color rgba="0.35 0.35 0.35 1" />
+					</material>
 			</visual>
 		</link>
@@ -36,4 +36,4 @@
 		 	accel_mean="${accel_mean}" accel_stddev="${accel_stddev}" accel_bias_mean="${accel_bias_mean}"
 		 	accel_bias_stddev="${accel_bias_stddev}"/>
-	</xacro:macro>
+		</xacro:macro>
 </robot>

Commit message: [cleanup] Removed the parameters for setting the imu properties

File: urdfs/sensors/kvh_1775_imu.urdf.xacro (robot description, xacro)
@@ -4,6 +4,5 @@
 	<!-- ============================ IMU KVH 1775 ============================== -->
 	<!-- The xacro macro xacro:kvh_1775_imu: imu frame -->
-	<xacro:macro name="kvh_1775_imu" params="parent *origin imu_name imu_topic update_rate
-		rate_mean rate_stddev rate_bias_mean rate_bias_stddev accel_mean accel_stddev accel_bias_mean accel_bias_stddev">
+	<xacro:macro name="kvh_1775_imu" params="parent *origin imu_name imu_topic update_rate">
 		<!-- Joint -->
 		<joint name="${imu_name}_joint" type="fixed">

File: urdfs/sensors/microstrain_3dmgx325_imu.urdf.xacro (robot description, xacro)
@@ -4,6 +4,5 @@
 	<!-- ============================ IMU microstrain ============================== -->
 	<!-- The xacro macro xacro:microstrain_3dmgx325_imu: imu frame -->
-	<xacro:macro name="microstrain_3dmgx325_imu" params="parent *origin imu_name imu_topic update_rate
-		rate_mean rate_stddev rate_bias_mean rate_bias_stddev accel_mean accel_stddev accel_bias_mean accel_bias_stddev">
+	<xacro:macro name="microstrain_3dmgx325_imu" params="parent *origin imu_name imu_topic update_rate">
 		<!-- Joint -->
 		<joint name="${imu_name}_joint" type="fixed">

Commit message: [cleanup] Improved the spacing of code lines

File: urdfs/sensors/kvh_1775_imu.urdf.xacro (robot description, xacro)
@@ -14,17 +14,17 @@
 		<link name="${imu_name}">
 			<inertial>
-                <origin xyz="-0.001  0.0005  -0.00405"/>
-                <mass value="0.7"/>
+				<origin xyz="-0.001  0.0005  -0.00405"/>
+				<mass value="0.7"/>
 				<inertia ixx="0.0" iyy="0.0" izz="0.0" ixy="0.0" ixz="0.0" iyz="0.0"/>
 			</inertial>
 			<visual>
-                <origin xyz="0.0213 -0.0029 -0.00155" rpy="0 0 0"/>
-                <origin xyz="0.0 0.0 0.0" rpy="0 0 0"/>
+				<origin xyz="0.0213 -0.0029 -0.00155" rpy="0 0 0"/>
+				<origin xyz="0.0 0.0 0.0" rpy="0 0 0"/>
 				<geometry>
 					<cylinder radius="0.0482" length="0.0737" />
 				</geometry>
-					<material name="aluminium">
-						<color rgba="0.35 0.35 0.35 1" />
-					</material>
+				<material name="aluminium">
+					<color rgba="0.35 0.35 0.35 1" />
+				</material>
 			</visual>
 		</link>

Commit message: updated KVH and Microstrain IMUs to have all the proper reference frames

File: urdfs/sensors/kvh_1775_imu.urdf.xacro (robot description, xacro)
@@ -2,25 +2,118 @@
 <robot xmlns:xacro="http://ros.org/wiki/xacro">
 	<xacro:include filename="$(find sensors_description)/urdfs/sensors/imu.gazebo.xacro"/>
-	<!-- ============================ IMU KVH 1775 ============================== -->
-	<!-- The xacro macro xacro:kvh_1775_imu: imu frame -->
+        <!-- ============================ IMU KVH 1775 ========================
+         The xacro macro xacro:kvh_1775_imu describes the KVH 1775 IMU,
+         together with its frames of reference.
+         The IMU has three axes oriented along the diagonal of the mounting
+         screws at the bottom, as described at page 6 of the technical manual.
+         These axes have three different origins for the sensing points, one
+         per axis. Therefore, we define a common origin which is located at the
+         average of these three. For completeness, we include the three exact
+         axes as well. -->
 	<xacro:macro name="kvh_1775_imu" params="parent *origin imu_name imu_topic update_rate">
-		<!-- Joint -->
-		<joint name="${imu_name}_joint" type="fixed">
+                <!-- Joint connecting the mount point of the IMU to the robot -->
+                <joint name="${imu_name}_mount_joint" type="fixed">
 			<xacro:insert_block name="origin"/>
 			<parent link="${parent}" />
-			<child link="${imu_name}"/>
+                        <child link="${imu_name}_mount"/>
 		</joint>
+                <!-- Fake joint connecting the mount point of the IMU to the
+                     average sensing frame of the IMU -->
+                <joint name="${imu_name}_joint" type="fixed">
+                                        <origin xyz="-0.017066667 -0.013 0.038366667" rpy="0 0 0"/>
+                    <parent link="${imu_name}_mount" />
+                    <child link="${imu_name}"/>
+                </joint>
+                <!-- Fake joint connecting the mount point of the IMU to
+                     the sensing point for the x-axis -->
+                <joint name="${imu_name}_sensing_point_x_joint" type="fixed">
+                    <origin xyz="0 -0.0263 0.0336" rpy="0 0 0"/>
+                    <parent link="${imu_name}_mount" />
+                    <child link="${imu_name}_sensing_point_x"/>
+                </joint>
+                <!-- Fake joint connecting the mount point of the IMU to
+                     the sensing point for the x-axis -->
+                <joint name="${imu_name}_sensing_point_y_joint" type="fixed">
+                    <origin xyz="-0.0256 -0.0121 0.0372" rpy="0 0 0"/>
+                    <parent link="${imu_name}_mount" />
+                    <child link="${imu_name}_sensing_point_y"/>
+                </joint>
+                <!-- Fake joint connecting the mount point of the IMU to
+                the sensing point for the x-axis -->
+                <joint name="${imu_name}_sensing_point_z_joint" type="fixed">
+                    <origin xyz="-0.0256 -0.0006 0.0443" rpy="0 0 0"/>
+                    <parent link="${imu_name}_mount" />
+                    <child link="${imu_name}_sensing_point_z"/>
+                </joint>
+                <!-- Fake link expressing the average sensing reference frame -->
+                <link name="${imu_name}">
+                    <inertial>
+                        <mass value="0.000" />
+                        <origin xyz="0 0 0" rpy="0 0 0"/>
+                        <inertia ixx="0.00" ixy="0.0" ixz="0.0" iyy="0.00" iyz="0.0" izz="0.00"/>
+                    </inertial>
+                    <visual>
+                        <!-- fake visual to let URDF parser happy -->
+                        <geometry>
+                                <sphere radius="0.0005"/>
+                        </geometry>
+                    </visual>
+                </link>
+                <!-- Fake link exactly located at the sensing point for the x-axis -->
+                <link name="${imu_name}_sensing_point_x">
+                    <inertial>
+                        <mass value="0.000" />
+                        <origin xyz="0 0 0" rpy="0 0 0"/>
+                        <inertia ixx="0.00" ixy="0.0" ixz="0.0" iyy="0.00" iyz="0.0" izz="0.00"/>
+                    </inertial>
+                    <visual>
+                        <!-- fake visual to let URDF parser happy -->
+                        <geometry>
+                                <sphere radius="0.0005"/>
+                        </geometry>
+                    </visual>
+                </link>
+                <!-- Fake link expressing the exact sensing point for the y-axis -->
+                <link name="${imu_name}_sensing_point_y">
+                    <inertial>
+                        <mass value="0.000" />
+                        <origin xyz="0 0 0" rpy="0 0 0"/>
+                        <inertia ixx="0.00" ixy="0.0" ixz="0.0" iyy="0.00" iyz="0.0" izz="0.00"/>
+                    </inertial>
+                    <visual>
+                        <!-- fake visual to let URDF parser happy -->
+                        <geometry>
+                                <sphere radius="0.0005"/>
+                        </geometry>
+                    </visual>
+                </link>
+                <!-- Fake link expressing the exact sensing point for the z-axis -->
+                <link name="${imu_name}_sensing_point_z">
+                    <inertial>
+                        <mass value="0.000" />
+                        <origin xyz="0 0 0" rpy="0 0 0"/>
+                        <inertia ixx="0.00" ixy="0.0" ixz="0.0" iyy="0.00" iyz="0.0" izz="0.00"/>
+                    </inertial>
+                    <visual>
+                        <!-- fake visual to let URDF parser happy -->
+                        <geometry>
+                                <sphere radius="0.0005"/>
+                        </geometry>
+                    </visual>
+                </link>
 		<!-- Link -->
-		<link name="${imu_name}">
+                <link name="${imu_name}_mount">
 			<inertial>
-				<origin xyz="-0.001  0.0005  -0.00405"/>
-				<mass value="0.7"/>
-				<inertia ixx="0.0" iyy="0.0" izz="0.0" ixy="0.0" ixz="0.0" iyz="0.0"/>
+                                <!-- CoM from technical document, rotated by pi/4 -->
+                                <origin xyz="-0.001697056  -0.001414214  0.0328"/>
+                                <mass value="0.69"/>
+                                <!-- izz = 0.5 * 0.69 * (88.9 / 2 / 1000)^2 -->
+                                <!-- ixx = iyy = 1/12*0.69*(3*(88.9/2000)^2+(73.7/1000)^2) -->
+                                <inertia ixx="0.000653148" iyy="0.000653148" izz="0.000681652" ixy="0.0" ixz="0.0" iyz="0.0"/>
 			</inertial>
 			<visual>
-				<origin xyz="0.0213 -0.0029 -0.00155" rpy="0 0 0"/>
 				<origin xyz="0.0 0.0 0.0" rpy="0 0 0"/>
 				<geometry>
-					<cylinder radius="0.0482" length="0.0737" />
+					<mesh filename="package://sensors_description/meshes/sensors/kvh_1775.dae" scale="1 1 1" />
 				</geometry>
 				<material name="aluminium">

File: urdfs/sensors/microstrain_3dmgx425_imu.urdf.xacro (robot description, xacro)
@@ -5,26 +5,44 @@
 	<!-- ============================ IMU microstrain ============================== -->
 	<!-- The xacro macro xacro:microstrain_3dmgx425_imu: imu frame -->
+        <!-- see Fig. 34 page 61 of Technical manual -->
 	<xacro:macro name="microstrain_3dmgx425_imu" params="parent *origin imu_name imu_topic update_rate">
 		<!-- Joint -->
 		<joint name="${imu_name}_joint" type="fixed">
-			<xacro:insert_block name="origin"/>
-			<parent link="${parent}" />
-			<child link="${imu_name}"/>
+                        <origin xyz="0.00485 0 0.0045" rpy="0.0 ${-PI} 0.0"/>
+                        <parent link="${imu_name}_mount" />
+                        <child link="${imu_name}"/>
 		</joint>
+                <joint name="${imu_name}_mount_joint" type="fixed">
+                        <xacro:insert_block name="origin"/>
+                        <parent link="${parent}" />
+                        <child link="${imu_name}_mount"/>
+                </joint>
+                <link name="${imu_name}_mount">
+                <inertial>
+                    <origin xyz="-0.00020  0.00010  0.00110"/>
+                    <mass value="0.018"/>
+                    <inertia ixx="0.0" iyy="0.0" izz="0.0" ixy="0.0" ixz="0.0" iyz="0.0"/>
+                </inertial>
+                <visual>
+                        <origin xyz="0.0 0.0 0.00555" rpy="0 0 0"/>
+                        <geometry>
+                                <box size="0.0329 0.0244 0.0111" />
+                        </geometry>
+                        <material name="black">
+                                <color rgba="0 0 0 0.9"/>
+                        </material>
+                </visual>
+                </link>
 		<!-- Link -->
 		<link name="${imu_name}">
 			<inertial>
-				<origin xyz="-0.00020  0.00010  0.00110"/>
-				<mass value="0.018"/>
+                                <origin xyz="0.0  0.0  0.0"/>
+                                <mass value="0.00"/>
 				<inertia ixx="0.0" iyy="0.0" izz="0.0" ixy="0.0" ixz="0.0" iyz="0.0"/>
 			</inertial>
 			<visual>
-				<origin xyz="0.00485 0 -0.00105" rpy="0 0 0"/>
 				<geometry>
-					<box size="0.0329 0.0244 0.0111" />
+                                        <sphere radius="0.0005" />
 				</geometry>
-				<material name="black">
-					<color rgba="0 0 0 0.9"/>
-				</material>
 			</visual>
 		</link>
