Commit message: [config] Using the same inertia properties for both microstrain IMUs

File: urdfs/sensors/microstrain_3dmgx325_imu.urdf.xacro (robot description, xacro)
@@ -19,8 +19,11 @@
 			</inertial>
 			<visual>
-				<origin xyz="0 0 0" rpy="0 0 0"/>
+				<origin xyz="0.00485 0 -0.00105" rpy="0 0 0"/>
 				<geometry>
-					<box size="0.02 0.02 0.02" />
+					<box size="0.0329 0.0244 0.0111" />
 				</geometry>
+				<material name="black">
+					<color rgba="0 0 0 0.9"/>
+				</material>
 			</visual>
 		</link>

Commit message: removed mass from  microstrain that is not accounted in robcogen!!!!!

File: urdfs/sensors/microstrain_3dmgx325_imu.urdf.xacro (robot description, xacro)
@@ -15,5 +15,5 @@
 			<inertial>
 				<origin xyz="-0.00020  0.00010  0.00110"/>
-				<mass value="0.018"/>
+                                <mass value="0.001"/>
 				<inertia ixx="0.0" iyy="0.0" izz="0.0" ixy="0.0" ixz="0.0" iyz="0.0"/>
 			</inertial>

File: urdfs/sensors/microstrain_3dmgx425_imu.urdf.xacro (robot description, xacro)
@@ -21,5 +21,5 @@
                 <inertial>
                     <origin xyz="-0.00020  0.00010  0.00110"/>
-                    <mass value="0.018"/>
+                    <mass value="0.001"/>
                     <inertia ixx="0.0" iyy="0.0" izz="0.0" ixy="0.0" ixz="0.0" iyz="0.0"/>
                 </inertial>
@@ -38,5 +38,5 @@
 			<inertial>
                                 <origin xyz="0.0  0.0  0.0"/>
-                                <mass value="0.00"/>
+                                <mass value="0.001"/>
 				<inertia ixx="0.0" iyy="0.0" izz="0.0" ixy="0.0" ixz="0.0" iyz="0.0"/>
 			</inertial>
