Commit message: Multisense fixed hokuyo link mesh and position based on wpi drc stuff

File: urdfs/sensors/multisense_sl.urdf.xacro (robot description, xacro)
@@ -60,10 +60,12 @@
   <link name="hokuyo_link">
     <inertial>
-      <origin xyz="0.012428 0.0004084 -0.0041835" rpy="0 0 0" />
-      <mass value="0.057664" />
+      <origin xyz="0.032428 0.0004084 -0.0041835" rpy="0 0 0" />
+      <mass value="0.057654" />
       <inertia iyy="4.2412E-05" ixy="4.9927E-08" iyz="-9.8165E-09" ixx="3.7174E-05" ixz="1.1015E-05" izz="4.167E-05" />
     </inertial>
     <visual>
-      <origin xyz="-.03 -.1 0" rpy="-1.9179632679 -1.57079632679 0" />
+      <!--origin xyz="0.065774 -0.001163 -0.08809" rpy="0 0 0" /-->
+      <!--origin xyz="0.045 -0.001163 -0.08809" rpy="-0.314 0 0" /-->
+      <origin xyz="0.045 -0.0261018277 -0.08342369" rpy="-0.314 0 0" />
       <geometry>
         <mesh filename="package://multisense_description/meshes/head_camera.dae" />
@@ -74,4 +76,10 @@
     </visual>
   <collision>
+    <origin xyz="0.01885 0 -0.02119" rpy="0 0 0" />
+    <geometry>
+      <box size="0.08 0.06 0.04238"/>
+    </geometry>
+  </collision>
+  <collision>
     <origin xyz="0.03 0 0.0235" rpy="0 0 0" />
     <geometry>

Commit message: [cleanup] Cosmetic changes

File: urdfs/sensors/multisense_sl.urdf.xacro (robot description, xacro)
@@ -2,214 +2,216 @@
 <robot xmlns:xacro="http://ros.org/wiki/xacro">
 <xacro:macro name="multisense_sl" params="parent *origin prefix" >
-  <joint name="${parent}_head_root_joint" type="fixed">
-    <insert_block name="origin"/>
-    <parent link="${parent}"/>
-    <child link="head_root"/>
-  </joint>
-  <!-- Head Link Simplified Collision Mesh -->
-  <link name="head_root"/>
-  <joint name="head_root_joint" type="fixed">
-    <parent link="head_root"/>
-    <child link="head"/>
-  </joint>
-  <link name="head">
-    <inertial>
-      <origin xyz="-0.075493 3.3383E-05 0.02774" rpy="0 0 0" />
-      <mass value="1.4199" />
-      <inertia iyy="0.0041178" ixy="-1.5797E-06" iyz="-6.8415E-07" ixx="0.0039688" ixz="-0.00089293" izz="0.0035243" />
-    </inertial>
-    <visual>
-      <origin xyz="0 0  0" rpy="0 0 0" />
-      <geometry>
-          <mesh filename="package://multisense_description/meshes/head.dae" />
-      </geometry>
-      <material name="">
-        <color rgba="0.9098 0.44314 0.031373 1" />
-      </material>
-    </visual>
-  <collision>
-    <origin xyz="-0.0503 0 -0.00195" rpy="0 0 0" />
-    <geometry>
-      <box size="0.1311 0.12 0.0591"/>
-    </geometry>
-  </collision>
-  </link>
-  <joint name="${prefix}/left_camera_optical_joint" type="continuous">
-    <parent link="${prefix}/left_camera_optical_frame" />
-    <child link="${prefix}/motor" />
-  </joint>
-  <link name="${prefix}/motor"/>
-  <link name="${prefix}/spindle"/>
-  <joint name="${prefix}/motor_joint" type="continuous">
-    <parent link="${prefix}/motor" />
-    <child link="${prefix}/spindle" />
-    <axis xyz="0 0 1" />
-  </joint>
-  <joint name="{prefix}/spindle_joint" type="continuous">
-    <parent link="${prefix}/spindle" />
-    <child link="${prefix}/hokuyo_link" />
-  </joint>
-  <link name="${prefix}/hokuyo_link">
-    <inertial>
-      <origin xyz="0.012428 0.0004084 -0.0041835" rpy="0 0 0" />
-      <mass value="0.057664" />
-      <inertia iyy="4.2412E-05" ixy="4.9927E-08" iyz="-9.8165E-09" ixx="3.7174E-05" ixz="1.1015E-05" izz="4.167E-05" />
-    </inertial>
-    <visual>
-      <origin xyz="-.03 -.1 0" rpy="-1.9179632679 -1.57079632679 0" />
-      <geometry>
-        <mesh filename="package://multisense_description/meshes/head_camera.dae" />
-      </geometry>
-      <material name="">
-        <color rgba="0.72941 0.35686 0.023529 1" />
-      </material>
-    </visual>
-  <collision>
-    <origin xyz="0.03 0 0.0235" rpy="0 0 0" />
-    <geometry>
-      <cylinder radius="0.024425" length="0.047"/>
-    </geometry>
-  </collision>
-  </link>
-  <link name="${prefix}/head_hokuyo_frame"/>
-  <joint name="${prefix}/head_hokuyo_frame_joint" type="fixed">
-    <!--
-     This transform accounts for the fact ROS expects laser data in the x forward,
-     y left, z up frame and the calibraton has the data in x left, y up, z forward.
-     Thus a roll of -90 * a pitch of -90 will make the appropriate transform. Note
-     Roll and pitch are both with respect to the origional x left, y up, z forward frame
-     -->
-    <origin xyz="0 0 0" rpy="-1.57079632679 -1.57079632679 0.0" />
-    <parent link="${prefix}/hokuyo_link" />
-    <child link="${prefix}/head_hokuyo_frame"/>
-  </joint>
-  <!-- Stereo Camera -->
-  <joint name="{prefix}/left_camera_frame_joint" type="fixed">
-    <!-- optical frame collocated with tilting DOF -->
-    <origin xyz="0.0 0.035 -0.002"/>
-    <parent link="head"/>
-    <child link="${prefix}/left_camera_frame"/>
-  </joint>
-  <link name="${prefix}/left_camera_frame">
-    <inertial>
-      <mass value="0.1" />
-      <origin xyz="0 0 0" />
-      <inertia ixx="0.001"  ixy="0.0"  ixz="0.0" iyy="0.001"  iyz="0.0" izz="0.001" />
-    </inertial>
-  </link>
-  <joint name="{prefix}/left_camera_optical_frame_joint" type="fixed">
-    <origin xyz="0 0 0" rpy="-1.57079632679 0.0 -1.57079632679" />
-    <parent link="${prefix}/left_camera_frame" />
-    <child link="${prefix}/left_camera_optical_frame"/>
-  </joint>
-  <link name="${prefix}/left_camera_optical_frame"/>
-  <joint name="${prefix}/right_camera_frame_joint" type="fixed">
-    <origin xyz="0.0 -0.035 -0.002"/>
-    <parent link="head"/>
-    <child link="${prefix}/right_camera_frame"/>
-  </joint>
-  <link name="${prefix}/right_camera_frame">
-    <inertial>
-      <mass value="0.1" />
-      <origin xyz="0 0 0" />
-      <inertia ixx="0.001"  ixy="0.0"  ixz="0.0" iyy="0.001"  iyz="0.0" izz="0.001" />
-    </inertial>
-  </link>
-  <joint name="${prefix}/right_camera_optical_frame_joint" type="fixed">
-    <origin xyz="0 0 0" rpy="-1.5708 0.0 -1.5708" />
-    <parent link="${prefix}/right_camera_frame" />
-    <child link="${prefix}/right_camera_optical_frame"/>
-  </joint>
-  <link name="${prefix}/right_camera_optical_frame"/>
-  <joint name="${prefix}/center_top_led_frame_joint" type="fixed">
-    <origin xyz="0.01125 0.0 0.0105"/>
-    <parent link="head"/>
-    <child link="${prefix}/center_top_led_frame"/>
-  </joint>
-  <link name="${prefix}/center_top_led_frame">
-    <inertial>
-      <mass value="0.1"/>
-      <origin xyz="0 0 0"/>
-      <inertia ixx="0.001" ixy="0.0" ixz="0.0" iyy="0.001" iyz="0.0" izz="0.001"/>
-    </inertial>
-  </link>
-  <joint name="${prefix}/center_bottom_led_frame_joint" type="fixed">
-    <origin xyz="0.01125 0.0 -0.0155"/>
-    <parent link="head"/>
-    <child link="${prefix}/center_bottom_led_frame"/>
-  </joint>
-  <link name="${prefix}/center_bottom_led_frame">
-    <inertial>
-      <mass value="0.1"/>
-      <origin xyz="0 0 0"/>
-      <inertia ixx="0.001" ixy="0.0" ixz="0.0" iyy="0.001" iyz="0.0" izz="0.001"/>
-    </inertial>
-  </link>
-  <joint name="${prefix}/left_led_frame_joint" type="fixed">
-    <origin xyz="-0.01443 0.07452 0.050346" rpy="0 -0.15 0.53"/>
-    <parent link="head"/>
-    <child link="${prefix}/left_led_frame"/>
-  </joint>
-  <link name="${prefix}/left_led_frame">
-    <inertial>
-      <mass value="0.1"/>
-      <origin xyz="0 0 0"/>
-      <inertia ixx="0.001" ixy="0.0" ixz="0.0" iyy="0.001" iyz="0.0" izz="0.001"/>
-    </inertial>
-  </link>
-  <joint name="{prefix}/right_led_frame_joint" type="fixed">
-    <origin xyz="-0.01443 -0.07452 0.050346" rpy="0 -0.15 -0.53"/>
-    <parent link="head"/>
-    <child link="${prefix}/right_led_frame"/>
-  </joint>
-  <link name="${prefix}/right_led_frame">
-    <inertial>
-      <mass value="0.1"/>
-      <origin xyz="0 0 0"/>
-      <inertia ixx="0.001" ixy="0.0" ixz="0.0" iyy="0.001" iyz="0.0" izz="0.001"/>
-    </inertial>
-  </link>
-  <!-- IMU Frames, Mag/Accel and Gyro -->
-  <!-- Include transfrom to the left_camera_frame (shift in -.035mm in X and -.002mm in Z) -->
-  <!-- imu link -->
-  <link name="${prefix}/head_imu_link">
-    <inertial>
-      <mass value="1e-5" />
-      <!-- collocate with parent link and remove mass from it -->
-      <origin xyz="-0.122993 0.035033383 0.02774" rpy="0 0 0" />
-      <inertia ixx="1e-6" ixy="0" ixz="0" iyy="1e-6" iyz="0" izz="1e-6" />
-    </inertial>
-    <visual>
-      <origin rpy="0 0 0" xyz="0 0 0"/>
-      <geometry>
-        <box size="0.01 0.01 0.01"/>
-      </geometry>
-    </visual>
-  </link>
-  <joint name="${prefix}/head_imu_joint" type="fixed">
-    <parent link="head"/>
-    <child link="${prefix}/head_imu_link"/>
-    <!-- putting it at the same z-level as the stereo -->
-    <origin xyz="-0.0475 0.035 0.0" rpy="0 0 0"/>
-  </joint>
-  <xacro:multisense_sl_sensor prefix="hyq"/>
-  <link name="${prefix}/accel"/>
-  <joint name="${prefix}/accel_joint" type="fixed">
-    <origin xyz="-.0475 .0302 -.00275" rpy="0 1.5707 0"/>
-    <parent link="head_root"/>
-    <child link="${prefix}/accel"/>
-  </joint>
-  <link name="${prefix}/mag"/>
-  <joint name="${prefix}/mag_joint" type="fixed">
-    <origin xyz="-.0475 .0302 -.00275" rpy="0 1.5707 0"/>
-    <parent link="head_root"/>
-    <child link="${prefix}/mag"/>
-  </joint>
-  <link name="${prefix}/gyro"/>
-  <joint name="${prefix}/gyro_joint" type="fixed">
-    <origin xyz="-.0476 .0388 -.00075" rpy="1.5707 3.14159 1.5707 "/>
-    <parent link="head_root"/>
-    <child link="${prefix}/gyro"/>
-  </joint>
+	<joint name="${parent}_head_root_joint" type="fixed">
+		<insert_block name="origin"/>
+		<parent link="${parent}"/>
+		<child link="head_root"/>
+	</joint>
+	<!-- Multisense joints -->
+	<link name="head_root"/>
+	<joint name="head_root_joint" type="fixed">
+		<parent link="head_root"/>
+		<child link="head"/>
+	</joint>
+	<joint name="${prefix}/left_camera_optical_joint" type="continuous">
+		<parent link="${prefix}/left_camera_optical_frame" />
+		<child link="${prefix}/motor" />
+	</joint>
+	<joint name="${prefix}/motor_joint" type="continuous">
+		<parent link="${prefix}/motor" />
+		<child link="${prefix}/spindle" />
+		<axis xyz="0 0 1" />
+	</joint>
+	<joint name="{prefix}/spindle_joint" type="continuous">
+		<parent link="${prefix}/spindle" />
+		<child link="${prefix}/hokuyo_link" />
+	</joint>
+	<joint name="${prefix}/head_hokuyo_frame_joint" type="fixed">
+		<!--
+		This transform accounts for the fact ROS expects laser data in the x forward,
+		y left, z up frame and the calibraton has the data in x left, y up, z forward.
+		Thus a roll of -90 * a pitch of -90 will make the appropriate transform. Note
+		Roll and pitch are both with respect to the origional x left, y up, z forward frame
+		-->
+		<origin xyz="0 0 0" rpy="-1.57079632679 -1.57079632679 0.0" />
+		<parent link="${prefix}/hokuyo_link" />
+		<child link="${prefix}/head_hokuyo_frame"/>
+	</joint>
+	<!-- Stereo Camera -->
+	<joint name="{prefix}/left_camera_frame_joint" type="fixed">
+		<!-- optical frame collocated with tilting DOF -->
+		<origin xyz="0.0 0.035 -0.002"/>
+		<parent link="head"/>
+		<child link="${prefix}/left_camera_frame"/>
+	</joint>
+	<joint name="{prefix}/left_camera_optical_frame_joint" type="fixed">
+		<origin xyz="0 0 0" rpy="-1.57079632679 0.0 -1.57079632679" />
+		<parent link="${prefix}/left_camera_frame" />
+		<child link="${prefix}/left_camera_optical_frame"/>
+	</joint>
+	<joint name="${prefix}/right_camera_frame_joint" type="fixed">
+		<origin xyz="0.0 -0.035 -0.002"/>
+		<parent link="head"/>
+		<child link="${prefix}/right_camera_frame"/>
+	</joint>
+	<joint name="${prefix}/right_camera_optical_frame_joint" type="fixed">
+		<origin xyz="0 0 0" rpy="-1.5708 0.0 -1.5708" />
+		<parent link="${prefix}/right_camera_frame" />
+		<child link="${prefix}/right_camera_optical_frame"/>
+	</joint>
+	<joint name="${prefix}/center_top_led_frame_joint" type="fixed">
+		<origin xyz="0.01125 0.0 0.0105"/>
+		<parent link="head"/>
+		<child link="${prefix}/center_top_led_frame"/>
+	</joint>
+	<joint name="${prefix}/center_bottom_led_frame_joint" type="fixed">
+		<origin xyz="0.01125 0.0 -0.0155"/>
+		<parent link="head"/>
+		<child link="${prefix}/center_bottom_led_frame"/>
+	</joint>
+	<joint name="${prefix}/left_led_frame_joint" type="fixed">
+		<origin xyz="-0.01443 0.07452 0.050346" rpy="0 -0.15 0.53"/>
+		<parent link="head"/>
+		<child link="${prefix}/left_led_frame"/>
+	</joint>
+	<joint name="{prefix}/right_led_frame_joint" type="fixed">
+		<origin xyz="-0.01443 -0.07452 0.050346" rpy="0 -0.15 -0.53"/>
+		<parent link="head"/>
+		<child link="${prefix}/right_led_frame"/>
+	</joint>
+	<joint name="${prefix}/head_imu_joint" type="fixed">
+		<parent link="head"/>
+		<child link="${prefix}/head_imu_link"/>
+		<!-- putting it at the same z-level as the stereo -->
+		<origin xyz="-0.0475 0.035 0.0" rpy="0 0 0"/>
+	</joint>
+	<joint name="${prefix}/accel_joint" type="fixed">
+		<origin xyz="-.0475 .0302 -.00275" rpy="0 1.5707 0"/>
+		<parent link="head_root"/>
+		<child link="${prefix}/accel"/>
+	</joint>
+	<joint name="${prefix}/mag_joint" type="fixed">
+		<origin xyz="-.0475 .0302 -.00275" rpy="0 1.5707 0"/>
+		<parent link="head_root"/>
+		<child link="${prefix}/mag"/>
+	</joint>
+	<joint name="${prefix}/gyro_joint" type="fixed">
+		<origin xyz="-.0476 .0388 -.00075" rpy="1.5707 3.14159 1.5707 "/>
+		<parent link="head_root"/>
+		<child link="${prefix}/gyro"/>
+	</joint>
+	<!-- Multisense links -->
+	<link name="head">
+		<inertial>
+			<origin xyz="-0.075493 3.3383E-05 0.02774" rpy="0 0 0" />
+			<mass value="1.4199" />
+			<inertia iyy="0.0041178" ixy="-1.5797E-06" iyz="-6.8415E-07" ixx="0.0039688" ixz="-0.00089293" izz="0.0035243" />
+		</inertial>
+		<visual>
+			<origin xyz="0 0 0" rpy="0 0 0" />
+			<geometry>
+				<mesh filename="package://multisense_description/meshes/head.dae" />
+			</geometry>
+			<material name="">
+				<color rgba="0.9098 0.44314 0.031373 1" />
+			</material>
+		</visual>
+		<collision>
+			<origin xyz="-0.0503 0 -0.00195" rpy="0 0 0" />
+			<geometry>
+				<box size="0.1311 0.12 0.0591"/>
+			</geometry>
+		</collision>
+	</link>
+	<link name="${prefix}/motor"/>
+	<link name="${prefix}/spindle"/>
+	<link name="${prefix}/hokuyo_link">
+		<inertial>
+			<origin xyz="0.012428 0.0004084 -0.0041835" rpy="0 0 0" />
+			<mass value="0.057664" />
+			<inertia iyy="4.2412E-05" ixy="4.9927E-08" iyz="-9.8165E-09" ixx="3.7174E-05" ixz="1.1015E-05" izz="4.167E-05" />
+		</inertial>
+		<visual>
+			<origin xyz="-.03 -.1 0" rpy="-1.9179632679 -1.57079632679 0" />
+			<geometry>
+				<mesh filename="package://multisense_description/meshes/head_camera.dae" />
+			</geometry>
+			<material name="">
+				<color rgba="0.72941 0.35686 0.023529 1" />
+			</material>
+		</visual>
+		<collision>
+			<origin xyz="0.03 0 0.0235" rpy="0 0 0" />
+			<geometry>
+				<cylinder radius="0.024425" length="0.047"/>
+			</geometry>
+		</collision>
+	</link>
+	<link name="${prefix}/head_hokuyo_frame"/>
+	<link name="${prefix}/left_camera_frame">
+		<inertial>
+			<mass value="0.1" />
+			<origin xyz="0 0 0" />
+			<inertia ixx="0.001"  ixy="0.0"  ixz="0.0" iyy="0.001"  iyz="0.0" izz="0.001" />
+		</inertial>
+	</link>
+	<link name="${prefix}/left_camera_optical_frame"/>
+	<link name="${prefix}/right_camera_frame">
+		<inertial>
+			<mass value="0.1" />
+			<origin xyz="0 0 0" />
+			<inertia ixx="0.001"  ixy="0.0"  ixz="0.0" iyy="0.001"  iyz="0.0" izz="0.001" />
+		</inertial>
+	</link>
+	<link name="${prefix}/right_camera_optical_frame"/>
+	<link name="${prefix}/center_top_led_frame">
+		<inertial>
+			<mass value="0.1"/>
+			<origin xyz="0 0 0"/>
+			<inertia ixx="0.001" ixy="0.0" ixz="0.0" iyy="0.001" iyz="0.0" izz="0.001"/>
+		</inertial>
+	</link>
+	<link name="${prefix}/center_bottom_led_frame">
+		<inertial>
+			<mass value="0.1"/>
+			<origin xyz="0 0 0"/>
+				<inertia ixx="0.001" ixy="0.0" ixz="0.0" iyy="0.001" iyz="0.0" izz="0.001"/>
+		</inertial>
+	</link>
+	<link name="${prefix}/left_led_frame">
+		<inertial>
+			<mass value="0.1"/>
+			<origin xyz="0 0 0"/>
+			<inertia ixx="0.001" ixy="0.0" ixz="0.0" iyy="0.001" iyz="0.0" izz="0.001"/>
+		</inertial>
+	</link>
+	<link name="${prefix}/right_led_frame">
+		<inertial>
+			<mass value="0.1"/>
+			<origin xyz="0 0 0"/>
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
Commit message: Adding fixed joint values from calibrated Multisense SL on hyq-green

File: urdfs/sensors/multisense_sl.urdf.xacro (robot description, xacro)
@@ -23,5 +23,5 @@
 		<parent link="${prefix}/left_camera_optical_frame" />
 		<child link="${prefix}/motor" />
-		<origin xyz="0.027 -0.097 -0.017" rpy="0. 0. 2." />
+		<origin xyz="0.027155533433 -0.0971753746271 -0.0172099247575" rpy="0.001972222 0.007801622 2.064951398" />
 	</joint>
 	<joint name="${prefix}/motor_joint" type="continuous">
@@ -33,5 +33,5 @@
 		<parent link="${prefix}/spindle" />
 		<child link="${prefix}/hokuyo_link" />
-		<origin xyz="0.001 0.01 0.0" rpy="0. 0. 0." />
+		<origin xyz="0.000662488571834 0.00996151566505 -0.00000718757200957" rpy="1.668656938 -1.547932514 3.043697136" />
 	</joint>
 	<joint name="${prefix}/head_hokuyo_frame_joint" type="fixed">

Commit message: Restored to continuous frame which has to be published by the sensor plugin

File: urdfs/sensors/multisense_sl.urdf.xacro (robot description, xacro)
@@ -20,8 +20,7 @@
 		<child link="head"/>
 	</joint>
-	<joint name="${prefix}/left_camera_optical_joint" type="fixed">
+	<joint name="${prefix}/left_camera_optical_joint" type="continuous">
 		<parent link="${prefix}/left_camera_optical_frame" />
 		<child link="${prefix}/motor" />
-		<origin xyz="0.027155533433 -0.0971753746271 -0.0172099247575" rpy="0.001972222 0.007801622 2.064951398" />
 	</joint>
 	<joint name="${prefix}/motor_joint" type="continuous">
@@ -30,8 +29,7 @@
 		<axis xyz="0 0 1" />
 	</joint>
-	<joint name="${prefix}/spindle_joint" type="fixed">
+	<joint name="${prefix}/spindle_joint" type="continuous">
 		<parent link="${prefix}/spindle" />
 		<child link="${prefix}/hokuyo_link" />
-		<origin xyz="0.000662488571834 0.00996151566505 -0.00000718757200957" rpy="1.668656938 -1.547932514 3.043697136" />
 	</joint>
 	<joint name="${prefix}/head_hokuyo_frame_joint" type="fixed">

Commit message: Add back the mass for the multisense

File: urdfs/sensors/multisense_sl.urdf.xacro (robot description, xacro)
@@ -113,6 +113,5 @@
 		<inertial>
 			<origin xyz="-0.075493 3.3383E-05 0.02774" rpy="0 0 0" />
-			<!--<mass value="1.4199" />-->
-			<mass value="0.001" />
+			<mass value="1.4199" />
 			<inertia iyy="0.0041178" ixy="-1.5797E-06" iyz="-6.8415E-07" ixx="0.0039688" ixz="-0.00089293" izz="0.0035243" />
 		</inertial>
