Commit message: Update for realsense

File: urdfs/sensors/realsense.gazebo.urdf.xacro (robot description, xacro)
@@ -4,10 +4,12 @@
 <gazebo>
 	<!--<plugin name="realsense_plugin" filename="libRealSensePlugin.so"/>-->
-	<plugin name="realsense_plugin" filename="librealsense_gazebo_plugin.so"/>
+	<plugin name="realsense_plugin" filename="librealsense_gazebo_plugin.so">
+		<prefix>${prefix}</prefix>
+	</plugin>
 </gazebo>
-<gazebo reference="${parent}_camera_joint" type="fixed">
+<gazebo reference="${prefix}/${parent}_camera_joint" type="fixed">
 	<pose frame="">0 0 0.015 0 0 0</pose>
 </gazebo>
-<gazebo reference="camera_link">
+<gazebo reference="${prefix}/camera_link">
 		<inertial>
 			<mass>0.0615752</mass>
@@ -73,5 +75,5 @@
 </gazebo>
 <gazebo reference="${prefix}/camera_fisheye_frame">
-		<sensor name="color" type="camera">
+		<sensor name="${prefix}color" type="camera">
 			<pose frame="">0 -0.046 0.004 0 0 0</pose>
 			<camera name="__default__">
@@ -87,5 +89,5 @@
 </gazebo>
 <gazebo reference="${prefix}/camera_left_ir_frame">
-		<sensor name="ired1" type="camera">
+		<sensor name="${prefix}ired1" type="camera">
 			<pose frame="">0 -0.06 0.004 0 0 0</pose>
 			<camera name="__default__">
@@ -101,5 +103,5 @@
 </gazebo>
 <gazebo reference="${prefix}/camera_right_ir_frame">
-		<sensor name="ired2" type="camera">
+		<sensor name="${prefix}ired2" type="camera">
 			<pose frame="">0 0.01 0.004 0 0 0</pose>
 			<camera name="__default__">
@@ -115,5 +117,5 @@
 </gazebo>
 <gazebo reference="${prefix}/camera_depth_frame">
-		<sensor name="depth" type="depth">
+		<sensor name="${prefix}depth" type="depth">
 			<pose frame="">0 -0.03 0.004 0 0 0</pose>
 			<camera name="__default__">

File: urdfs/sensors/realsense.urdf.xacro (robot description, xacro)
@@ -21,10 +21,10 @@
 <xacro:macro name="sensor_r430" params="parent *origin prefix">
 	<!-- camera body, with origin at bottom screw mount -->
-	<joint name="${parent}_camera_joint" type="fixed">
+	<joint name="${prefix}/${parent}_camera_joint" type="fixed">
 		<xacro:insert_block name="origin" />
 		<parent link="${parent}"/>
-		<child link="camera_link" />
+		<child link="${prefix}/camera_link" />
 	</joint>
-	<link name="camera_link">
+	<link name="${prefix}/camera_link">
 		<visual>
 			<origin xyz="0 ${-r430_cam_mount_from_center_offset} ${r430_cam_height/2}" rpy="${M_PI/2} 0 ${M_PI/2}"/>
@@ -51,5 +51,5 @@
 	<joint name="${prefix}/camera_depth_joint" type="fixed">
 		<origin xyz="${r430_cam_depth_px} ${r430_cam_depth_py} ${r430_cam_depth_pz}" rpy="0 0 0"/>
-		<parent link="camera_link"/>
+		<parent link="${prefix}/camera_link"/>
 		<child link="${prefix}/camera_depth_frame" />
 	</joint>
