Commit message: [cleanup] Using the same imu gazebo plugin for all the imus

File: urdfs/sensors/imu.gazebo.xacro (robot description, xacro)
@@ -1,7 +1,7 @@
 <?xml version="1.0"?>
 <robot xmlns:xacro="http://ros.org/wiki/xacro">
-	<xacro:macro name="microstrain_3dmgx325_imu_sensor" params="imu_name imu_topic update_rate
-		rate_mean rate_stddev rate_bias_mean rate_bias_stddev accel_mean accel_stddev accel_bias_mean accel_bias_stddev">
-		<gazebo>
+	<xacro:macro name="imu_sensor" params="imu_name imu_topic update_rate rate_mean rate_stddev
+		rate_bias_mean rate_bias_stddev accel_mean accel_stddev accel_bias_mean accel_bias_stddev">
+ 		<gazebo>
 			<plugin name="${imu_name}_controller" filename="libgazebo_ros_imu.so">
 				<alwaysOn>true</alwaysOn>
@@ -15,5 +15,5 @@
 			</plugin>
 		</gazebo>
-		<!-- Imu definition required for hardware interface of ros control -->
+		<!-- Imu definition required for HyQ2Max hardware interface of ros control -->
 		<gazebo reference="${imu_name}">
 			<sensor name="trunk_imu" type="imu">

File: urdfs/sensors/kvh_1775_imu.urdf.xacro (robot description, xacro)
@@ -1,5 +1,5 @@
 <?xml version="1.0"?>
 <robot xmlns:xacro="http://ros.org/wiki/xacro">
-    <!--xacro:include filename="$(find sensors_description)/urdfs/sensors/kvh_1775_imu.gazebo.xacro"/-->
+	<xacro:include filename="$(find sensors_description)/urdfs/sensors/imu.gazebo.xacro"/>
 	<!-- ============================ IMU KVH 1775 ============================== -->
 	<!-- The xacro macro xacro:kvh_1775_imu: imu frame -->
@@ -31,5 +31,5 @@
 		</link>
 		<!-- IMU definition -->
-		<xacro:kvh_1775_imu_sensor imu_name="${imu_name}" imu_topic="${imu_topic}"
+		<xacro:imu_sensor imu_name="${imu_name}" imu_topic="${imu_topic}"
 		 	update_rate="${update_rate}" rate_mean="${rate_mean}" rate_stddev="${rate_stddev}"
 		 	rate_bias_mean="${rate_bias_mean}" rate_bias_stddev="${rate_bias_stddev}"

File: urdfs/sensors/microstrain_3dmgx325_imu.urdf.xacro (robot description, xacro)
@@ -1,5 +1,5 @@
 <?xml version="1.0"?>
 <robot xmlns:xacro="http://ros.org/wiki/xacro">
-	<xacro:include filename="$(find sensors_description)/urdfs/sensors/microstrain_3dmgx325_imu.gazebo.xacro"/>
+	<xacro:include filename="$(find sensors_description)/urdfs/sensors/imu.gazebo.xacro"/>
 	<!-- ============================ IMU microstrain ============================== -->
 	<!-- The xacro macro xacro:microstrain_3dmgx325_imu: imu frame -->
@@ -27,5 +27,5 @@
 		</link>
 		<!-- IMU definition -->
-		<xacro:microstrain_3dmgx325_imu_sensor imu_name="${imu_name}" imu_topic="${imu_topic}"
+		<xacro:imu_sensor imu_name="${imu_name}" imu_topic="${imu_topic}"
 		 	update_rate="${update_rate}" rate_mean="${rate_mean}" rate_stddev="${rate_stddev}"
 		 	rate_bias_mean="${rate_bias_mean}" rate_bias_stddev="${rate_bias_stddev}"

File: urdfs/sensors/microstrain_3dmgx425_imu.urdf.xacro (robot description, xacro)
@@ -1,5 +1,15 @@
 <?xml version="1.0"?>
 <robot xmlns:xacro="http://ros.org/wiki/xacro">
-	<xacro:include filename="$(find sensors_description)/urdfs/sensors/microstrain_3dmgx425_imu.gazebo.xacro"/>
+	<xacro:include filename="$(find sensors_description)/urdfs/sensors/imu.gazebo.xacro"/>
+<!--
+	<property name="rate_mean" value="0" />
+	<property name="rate_stddev" value="2e-4" />
+	<property name="rate_bias_mean" value="0.00087" />
+	<property name="rate_bias_stddev" value="0.0000008" />
+	<property name="accel_mean" value="0" />
+	<property name="accel_stddev" value="1.7e-2" />
+	<property name="accel_bias_mean" value="0.002" />
+	<property name="accel_bias_stddev" value="0.001" />
+-->
 	<!-- ============================ IMU microstrain ============================== -->
 	<!-- The xacro macro xacro:microstrain_3dmgx425_imu: imu frame -->
@@ -30,5 +40,5 @@
 		</link>
 		<!-- IMU Gazebo plugin definition -->
-		<xacro:microstrain_3dmgx425_imu_sensor imu_name="${imu_name}" imu_topic="${imu_topic}"
+		<xacro:imu_sensor imu_name="${imu_name}" imu_topic="${imu_topic}"
 		 	update_rate="${update_rate}" rate_mean="${rate_mean}" rate_stddev="${rate_stddev}"
 		 	rate_bias_mean="${rate_bias_mean}" rate_bias_stddev="${rate_bias_stddev}"

Commit message: Add frame to xacro

File: urdfs/sensors/imu.gazebo.xacro (robot description, xacro)
@@ -2,5 +2,5 @@
 <robot xmlns:xacro="http://ros.org/wiki/xacro">
 	<xacro:macro name="imu_sensor" params="imu_name imu_topic update_rate rate_mean rate_stddev
-		rate_bias_mean rate_bias_stddev accel_mean accel_stddev accel_bias_mean accel_bias_stddev">
+                rate_bias_mean rate_bias_stddev accel_mean accel_stddev accel_bias_mean accel_bias_stddev frame_name">
  		<gazebo>
 			<plugin name="${imu_name}_controller" filename="libgazebo_ros_imu.so">
@@ -13,4 +13,5 @@
 				<rpyOffset>0 0 0</rpyOffset>
 				<serviceName>/${imu_name}_imu</serviceName>
+                                <frameName>${frame_name}</frameName>
 			</plugin>
 		</gazebo>

File: urdfs/sensors/kvh_1775_imu.urdf.xacro (robot description, xacro)
@@ -11,5 +11,5 @@
          average of these three. For completeness, we include the three exact
          axes as well. -->
-	<xacro:macro name="kvh_1775_imu" params="parent *origin imu_name imu_topic update_rate">
+        <xacro:macro name="kvh_1775_imu" params="parent *origin imu_name imu_topic update_rate frame_name">
                 <!-- Joint connecting the mount point of the IMU to the robot -->
                 <joint name="${imu_name}_mount_joint" type="fixed">
@@ -132,5 +132,7 @@
 		 	accel_stddev="${kvh_1775_acc_stddev}"
 			accel_bias_mean="${kvh_1775_acc_bias_mean}"
-		 	accel_bias_stddev="${kvh_1775_acc_bias_stddev}"/>
+                        accel_bias_stddev="${kvh_1775_acc_bias_stddev}"
+                        frame_name="${frame_name}"
+               />
 	</xacro:macro>
 </robot>

File: urdfs/sensors/microstrain_3dmgx425_imu.urdf.xacro (robot description, xacro)
@@ -6,5 +6,5 @@
 	<!-- The xacro macro xacro:microstrain_3dmgx425_imu: imu frame -->
         <!-- see Fig. 34 page 61 of Technical manual -->
-	<xacro:macro name="microstrain_3dmgx425_imu" params="parent *origin imu_name imu_topic update_rate">
+        <xacro:macro name="microstrain_3dmgx425_imu" params="parent *origin imu_name imu_topic update_rate frame_name">
 		<!-- Joint -->
 		<joint name="${imu_name}_joint" type="fixed">
@@ -57,5 +57,7 @@
 		 	accel_stddev="${microstrain_gx425_acc_stddev}"
 			accel_bias_mean="0.002"
-		 	accel_bias_stddev="0.001"/>
+                        accel_bias_stddev="0.001"
+                        frame_name="${frame_name}"
+                />
 	</xacro:macro>
 </robot>

Commit message: Add frame name to imus

File: urdfs/sensors/imu.gazebo.xacro (robot description, xacro)
@@ -1,6 +1,5 @@
 <?xml version="1.0"?>
 <robot xmlns:xacro="http://ros.org/wiki/xacro">
-	<xacro:macro name="imu_sensor" params="imu_name imu_topic update_rate rate_mean rate_stddev
-		rate_bias_mean rate_bias_stddev accel_mean accel_stddev accel_bias_mean accel_bias_stddev">
+	<xacro:macro name="imu_sensor" params="imu_name imu_topic frame_name update_rate rate_mean rate_stddev rate_bias_mean rate_bias_stddev accel_mean accel_stddev accel_bias_mean accel_bias_stddev">
  		<gazebo>
 			<plugin name="${imu_name}_controller" filename="libgazebo_ros_imu.so">
@@ -12,5 +11,6 @@
 				<xyzOffset>0 0 0</xyzOffset>
 				<rpyOffset>0 0 0</rpyOffset>
-				<serviceName>/${imu_name}_imu</serviceName>
+				<serviceName>/${imu_name}</serviceName>
+				<frameName>${frame_name}</frameName>
 			</plugin>
 		</gazebo>

File: urdfs/sensors/kvh_1775_imu.urdf.xacro (robot description, xacro)
@@ -11,5 +11,5 @@
          average of these three. For completeness, we include the three exact
          axes as well. -->
-	<xacro:macro name="kvh_1775_imu" params="parent *origin imu_name imu_topic update_rate">
+	<xacro:macro name="kvh_1775_imu" params="parent *origin imu_name imu_topic frame_name update_rate">
                 <!-- Joint connecting the mount point of the IMU to the robot -->
                 <joint name="${imu_name}_mount_joint" type="fixed">
@@ -123,5 +123,8 @@
 		</link>
 		<!-- IMU definition -->
-		<xacro:imu_sensor imu_name="${imu_name}" imu_topic="${imu_topic}"
+		<xacro:imu_sensor
+			imu_name="${imu_name}"
+			imu_topic="${imu_topic}"
+			frame_name="${frame_name}"
 		 	update_rate="${update_rate}"
 			rate_mean="${kvh_1775_vel_mean}"

File: urdfs/sensors/microstrain_3dmgx325_imu.urdf.xacro (robot description, xacro)
@@ -4,5 +4,5 @@
 	<!-- ============================ IMU microstrain ============================== -->
 	<!-- The xacro macro xacro:microstrain_3dmgx325_imu: imu frame -->
-	<xacro:macro name="microstrain_3dmgx325_imu" params="parent *origin imu_name imu_topic update_rate">
+	<xacro:macro name="microstrain_3dmgx325_imu" params="parent *origin imu_name imu_topic frame_name update_rate">
 		<!-- Joint -->
 		<joint name="${imu_name}_joint" type="fixed">
@@ -29,5 +29,8 @@
 		</link>
 		<!-- IMU Gazebo plugin definition -->
-		<xacro:imu_sensor imu_name="${imu_name}" imu_topic="${imu_topic}"
+		<xacro:imu_sensor
+			imu_name="${imu_name}"
+			imu_topic="${imu_topic}"
+			frame_name="${frame_name}"
 		 	update_rate="${update_rate}"
 			rate_mean="${microstrain_gx325_vel_mean}"

File: urdfs/sensors/microstrain_3dmgx425_imu.urdf.xacro (robot description, xacro)
@@ -6,5 +6,5 @@
 	<!-- The xacro macro xacro:microstrain_3dmgx425_imu: imu frame -->
         <!-- see Fig. 34 page 61 of Technical manual -->
-	<xacro:macro name="microstrain_3dmgx425_imu" params="parent *origin imu_name imu_topic update_rate">
+	<xacro:macro name="microstrain_3dmgx425_imu" params="parent *origin imu_name imu_topic frame_name update_rate">
 		<!-- Joint -->
 		<joint name="${imu_name}_joint" type="fixed">
@@ -48,5 +48,8 @@
 		</link>
 		<!-- IMU Gazebo plugin definition -->
-		<xacro:imu_sensor imu_name="${imu_name}" imu_topic="${imu_topic}"
+		<xacro:imu_sensor
+			imu_name="${imu_name}"
+			imu_topic="${imu_topic}"
+			frame_name="${frame_name}"
 		 	update_rate="${update_rate}"
 			rate_mean="${microstrain_gx425_vel_mean}"
