Commit message: Do not simulate lidar by default as it is slow

File: urdfs/sensors/vlp16.gazebo.urdf.xacro (robot description, xacro)
@@ -49,4 +49,5 @@
 				  <max_range>130.0</max_range>
 				  <gaussianNoise>0.008</gaussianNoise>
+				  <alwaysOn>false</alwaysOn>
 				</plugin>
 			</sensor>

File: urdfs/sensors/vlp16.urdf.xacro (robot description, xacro)
@@ -1,5 +1,6 @@
 <?xml version="1.0"?>
 <root xmlns:xacro="http://ros.org/wiki/xacro">
-<xacro:include filename="$(find sensors_description)/urdfs/sensors/vlp16.gazebo.urdf.xacro" />
+<xacro:property name="sim_lidar" value="false"/>
+  <xacro:include filename="$(find sensors_description)/urdfs/sensors/vlp16.gazebo.urdf.xacro" />
   <xacro:property name="M_PI" value="3.1415926535897931" />
   <xacro:macro name="VLP-16" params="*origin parent:=base_link name:=velodyne topic:=/velodyne_points hz:=10 lasers:=16 samples:=1875 collision_range:=0.3 min_range:=0.9 max_range:=130.0 noise:=0.008 min_angle:=-${M_PI} max_angle:=${M_PI} gpu:=false">
@@ -52,5 +53,7 @@
       </visual>
     </link>
+<xacro:if value="${sim_lidar}">
     <xacro:velodyne_sensor link_name="${name}" frame_name="${name}_base_link" lidar_name="${name}" />
+</xacro:if>
   </xacro:macro>
 </root>
