Commit message: Realsense debugging urdf

File: urdfs/sensors/d435_camera.gazebo.urdf.xacro (robot description, xacro)
@@ -1,5 +1,5 @@
 <?xml version="1.0"?>
 <robot xmlns:xacro="http://ros.org/wiki/xacro">
-<xacro:macro name="realsense_sensor" params="prefix">
+<xacro:macro name="d435_gazebo_camera" params="parent prefix">
 <gazebo>
 	<!--<plugin name="realsense_plugin" filename="libRealSensePlugin.so"/>-->
@@ -8,19 +8,68 @@
 	</plugin>
 </gazebo>
-<gazebo reference="${prefix}/${parent}_camera_joint" type="fixed">
-	<pose frame="">0 0 0.015 0 0 0</pose>
+<gazebo reference="${prefix}/camera_depth_frame">
+    <sensor name="${prefix}depth" type="depth">
+	    <camera name="__default__">
+		    <horizontal_fov>1.047</horizontal_fov>
+		    <image><width>640</width><height>480</height></image>
+		    <clip><near>0.1</near><far>100</far></clip>
+		    <noise><type>gaussian</type><mean>0.0</mean><stddev>0.007</stddev></noise>
+	    </camera>
+	    <always_on>1</always_on>
+	    <update_rate>60</update_rate>
+	    <visualize>1</visualize>
+    </sensor>
 </gazebo>
-<gazebo reference="${prefix}/camera_link">
+<gazebo reference="${prefix}/camera_left_ir_frame">
+    <sensor name="${prefix}ired1" type="camera">
+	    <camera name="__default__">
+		    <horizontal_fov>1.047</horizontal_fov>
+		    <image><width>640</width><height>480</height><format>L_INT8</format></image>
+		    <clip><near>0.1</near><far>100</far></clip>
+		    <noise><type>gaussian</type><mean>0.0</mean><stddev>0.007</stddev></noise>
+	    </camera>
+	    <always_on>0</always_on>
+	    <update_rate>60</update_rate>
+	    <visualize>0</visualize>
+    </sensor>
+</gazebo>
+<gazebo reference="${prefix}/camera_right_ir_frame">
+    <sensor name="${prefix}ired2" type="camera">
+	    <camera name="__default__">
+		    <horizontal_fov>1.047</horizontal_fov>
+		    <image><width>640</width><height>480</height><format>L_INT8</format></image>
+		    <clip><near>0.1</near><far>100</far></clip>
+		    <noise><type>gaussian</type><mean>0.0</mean><stddev>0.007</stddev></noise>
+	    </camera>
+	    <always_on>0</always_on>
+	    <update_rate>60</update_rate>
+	    <visualize>0</visualize>
+    </sensor>
+</gazebo>
+<gazebo reference="${prefix}/camera_color_frame">
+    <sensor name="${prefix}color" type="camera">
+	    <camera name="__default__">
+		    <horizontal_fov>1.047</horizontal_fov>
+		    <image><width>640</width><height>480</height><format>RGB_INT8</format></image>
+		    <clip><near>0.1</near><far>100</far></clip>
+		    <noise><type>gaussian</type><mean>0.0</mean><stddev>0.007</stddev></noise>
+	    </camera>
+	    <always_on>0</always_on>
+	    <update_rate>60</update_rate>
+	    <visualize>1</visualize>
+    </sensor>
+</gazebo>
+<!--gazebo reference="${prefix}/camera_link">
 		<inertial>
-			<mass>0.0615752</mass>
+			<mass>0.564</mass>
 			<inertia>
-				<ixx>9.108e-05</ixx>
+				<ixx>0.003881243</ixx>
 				<ixy>0</ixy>
 				<ixz>0</ixz>
-				<iyy>2.51e-06</iyy>
+				<iyy>0.000498940</iyy>
 				<iyz>0</iyz>
-				<izz>8.931e-05</izz>
+				<izz>0.003879257</izz>
 			</inertia>
-			<pose frame=''>0 0 0 0 -0 0</pose>
+			<pose frame=''>${d435_cam_mount_from_center_offset} ${-d435_cam_depth_py} 0 ${M_PI/2} 0 ${M_PI/2}</pose>
 		</inertial>
 		<self_collide>0</self_collide>
@@ -34,11 +83,11 @@
 				</mesh>
 			</geometry>
-		</visual>
-		<collision name='collision'>
+		</visual-->
+		<!--collision name='collision'>
 			<laser_retro>0</laser_retro>
 				<max_contacts>10</max_contacts>
-				<pose frame=''>0 0 0 0 -0 0</pose>
+				<pose frame=''>0 ${-d435_cam_depth_py} 0 0 0 0</pose>
 				<geometry>
-					<box><size>0.0078 0.130 0.0192</size></box>
+					<box><size>${d435_cam_depth} ${d435_cam_width} ${d435_cam_height}</size></box>
 				</geometry>
 			<surface>
@@ -73,8 +122,8 @@
 			</surface>
 		</collision>
-</gazebo>
-<gazebo reference="${prefix}/camera_fisheye_frame">
+</gazebo-->
+<!--gazebo reference="${prefix}/camera_color_frame">
 		<sensor name="${prefix}color" type="camera">
-			<pose frame="">0 -0.046 0.004 0 0 0</pose>
+			<pose frame=''>0 -0.046 0.004 0 0 0</pose>
 			<camera name="__default__">
 				<horizontal_fov>1.047</horizontal_fov>
@@ -90,5 +139,5 @@
 <gazebo reference="${prefix}/camera_left_ir_frame">
 		<sensor name="${prefix}ired1" type="camera">
-			<pose frame="">0 -0.06 0.004 0 0 0</pose>
+			<pose frame=''>0 -0.06 0.004 0 0 0</pose>
 			<camera name="__default__">
 				<horizontal_fov>1.047</horizontal_fov>
@@ -104,5 +153,5 @@
 <gazebo reference="${prefix}/camera_right_ir_frame">
 		<sensor name="${prefix}ired2" type="camera">
-			<pose frame="">0 0.01 0.004 0 0 0</pose>
+			<pose frame=''>0 0.01 0.004 0 0 0</pose>
 			<camera name="__default__">
 				<horizontal_fov>1.047</horizontal_fov>
@@ -118,5 +167,5 @@
 <gazebo reference="${prefix}/camera_depth_frame">
 		<sensor name="${prefix}depth" type="depth">
-			<pose frame="">0 -0.03 0.004 0 0 0</pose>
+			<pose frame=''>0 -0.03 0.004 0 0 0</pose>
 			<camera name="__default__">
 				<horizontal_fov>1.047</horizontal_fov>
@@ -129,5 +178,5 @@
 			<visualize>0</visualize>
 		</sensor>
-</gazebo>
+</gazebo-->
 </xacro:macro>
 </robot>

File: urdfs/sensors/d435_camera.urdf.xacro (robot description, xacro)
@@ -1,15 +1,112 @@
 <?xml version="1.0"?>
 <robot xmlns:xacro="http://ros.org/wiki/xacro">
-    <!--xacro:include filename="$(find realsense2_description)/urdf/_d435.urdf.xacro" /-->
-    <xacro:include filename="$(find sensors_description)/urdfs/sensors/realsense.urdf.xacro"/>
-    <xacro:include filename="$(find sensors_description)/urdfs/sensors/realsense.gazebo.urdf.xacro"/>
-    <xacro:macro name="d435_camera" params="parent prefix *origin">
-	<!--xacro:sensor_d435 parent="${parent}">
-	    <xacro:insert_block name="origin" />
-	</xacro:sensor_d435>
-	<xacro:realsense_sensor prefix="${prefix}"/-->
-	<xacro:sensor_r430 parent="${parent}" prefix="${prefix}">
-	    <xacro:insert_block name="origin" />
-	</xacro:sensor_r430>
-    </xacro:macro>
+<xacro:include filename="$(find sensors_description)/urdfs/sensors/d435_camera.gazebo.urdf.xacro"/>
+<xacro:property name="M_PI" value="3.1415926535897931" />
+<!-- The following values are approximate, and the camera node publishing TF values with actual calibrated camera extrinsic values -->
+<xacro:property name="d435_cam_depth_to_left_ir_offset" value="0.0"/>
+<xacro:property name="d435_cam_depth_to_right_ir_offset" value="-0.050"/>
+<xacro:property name="d435_cam_depth_to_color_offset" value="0.015"/>
+<!-- The following values model the aluminum peripherial case for the R430 camera, with the camera joint represented by the actual peripherial camera tripod mount -->
+<xacro:property name="d435_cam_width" value="0.090"/>
+<xacro:property name="d435_cam_height" value="0.025"/>
+<xacro:property name="d435_cam_depth" value="0.02505"/>
+<xacro:property name="d435_cam_mount_from_center_offset" value="0.0149"/>
+<!-- The following offset is relative the the physical D435 camera peripherial camera tripod mount -->
+<xacro:property name="d435_cam_depth_px" value="${d435_cam_mount_from_center_offset}"/>
+<xacro:property name="d435_cam_depth_py" value="0.0175"/>
+<xacro:property name="d435_cam_depth_pz" value="${d435_cam_height/2}"/>
+<material name="aluminum">
+	<color rgba="0.5 0.5 0.5 1"/>
+</material>
+<xacro:macro name="d435_camera" params="parent *origin prefix">
+    <!-- camera body, with origin at bottom screw mount -->
+    <joint name="${prefix}/${parent}camera_joint" type="fixed">
+      <xacro:insert_block name="origin" />
+      <parent link="${parent}"/>
+      <child link="${prefix}/camera_bottom_screw_frame" />
+    </joint>
+    <link name="${prefix}/camera_bottom_screw_frame"/>
+    <joint name="${prefix}/camera_link_joint" type="fixed">
+      <origin xyz="0 ${d435_cam_depth_py} ${d435_cam_depth_pz}" rpy="0 0 0"/>
+      <parent link="${prefix}/camera_bottom_screw_frame"/>
+      <child link="${prefix}/camera_link" />
+    </joint>
+	<link name="${prefix}/camera_link">
+		<visual>
+			<origin xyz="${d435_cam_mount_from_center_offset} ${-d435_cam_depth_py} 0" rpy="${M_PI/2} 0 ${M_PI/2}"/>
+			<geometry>
+				<!--box size="${d435_cam_width} ${d435_cam_height} ${d435_cam_depth}"/-->
+				<mesh filename="package://realsense2_description/meshes/d435.dae" />
+			</geometry>
+			<material name="aluminum"/>
+		</visual>
+		<collision>
+			<!--origin xyz="0.0 0.0 ${r430_cam_height/2}" rpy="0 0 0"/-->
+			<origin xyz="0 ${-d435_cam_depth_py} 0" rpy="0 0 0"/>
+			<geometry>
+				<box size="${d435_cam_depth} ${d435_cam_width} ${d435_cam_height}"/>
+			</geometry>
+		</collision>
+		<!-- The following are not reliable values, and should not be used for modeling -->
+		<inertial>
+			<mass value="0.564" />
+			<origin xyz="0 0 0" />
+			<inertia ixx="0.003881243" ixy="0.0" ixz="0.0" iyy="0.000498940" iyz="0.0" izz="0.003879257" />
+		</inertial>
+	</link>
+	<!-- camera depth joints and links -->
+	<joint name="${prefix}/camera_depth_joint" type="fixed">
+		<origin xyz="0 0 0" rpy="0 0 0"/>
+		<parent link="${prefix}/camera_link"/>
+		<child link="${prefix}/camera_depth_frame" />
+	</joint>
+	<link name="${prefix}/camera_depth_frame"/>
+	<joint name="${prefix}/camera_depth_optical_joint" type="fixed">
+		<origin xyz="0 0 0" rpy="${-M_PI/2} 0 ${-M_PI/2}" />
+		<parent link="${prefix}/camera_depth_frame" />
+		<child link="${prefix}/camera_depth_optical_frame" />
+	</joint>
+	<link name="${prefix}/camera_depth_optical_frame"/>
+	<!-- camera left IR joints and links -->
+	<joint name="${prefix}/camera_left_ir_joint" type="fixed">
+		<origin xyz="0 ${d435_cam_depth_to_left_ir_offset} 0" rpy="0 0 0" />
+		<parent link="${prefix}/camera_depth_frame" />
+		<child link="${prefix}/camera_left_ir_frame" />
+	</joint>
+	<link name="${prefix}/camera_left_ir_frame"/>
+	<joint name="${prefix}/camera_left_ir_optical_joint" type="fixed">
+		<origin xyz="0 0 0" rpy="${-M_PI/2} 0 ${-M_PI/2}" />
+		<parent link="${prefix}/camera_left_ir_frame" />
+		<child link="${prefix}/camera_left_ir_optical_frame" />
+	</joint>
+	<link name="${prefix}/camera_left_ir_optical_frame"/>
+	<!-- camera right IR joints and links -->
+	<joint name="${prefix}/camera_right_ir_joint" type="fixed">
+		<origin xyz="0 ${d435_cam_depth_to_right_ir_offset} 0" rpy="0 0 0" />
+		<parent link="${prefix}/camera_depth_frame" />
+		<child link="${prefix}/camera_right_ir_frame" />
+	</joint>
+	<link name="${prefix}/camera_right_ir_frame"/>
+	<joint name="${prefix}/camera_right_ir_optical_joint" type="fixed">
+		<origin xyz="0 0 0" rpy="${-M_PI/2} 0 ${-M_PI/2}" />
+		<parent link="${prefix}/camera_right_ir_frame" />
+		<child link="${prefix}/camera_right_ir_optical_frame" />
+	</joint>
+	<link name="${prefix}/camera_right_ir_optical_frame"/>
+	<!-- camera color joints and links -->
+	<joint name="${prefix}/camera_color_joint" type="fixed">
+		<origin xyz="0 ${d435_cam_depth_to_color_offset} 0" rpy="0 0 0" />
+		<parent link="${prefix}/camera_depth_frame" />
+		<child link="${prefix}/camera_color_frame" />
+	</joint>
+	<link name="${prefix}/camera_color_frame"/>
+	<joint name="${prefix}/camera_color_optical_joint" type="fixed">
+		<origin xyz="0 0 0" rpy="${-M_PI/2} 0 ${-M_PI/2}" />
+		<parent link="${prefix}/camera_color_frame" />
+		<child link="${prefix}/camera_color_optical_frame" />
+	</joint>
+	<link name="${prefix}/camera_color_optical_frame"/>
+	<!-- Gazebo realsense plugin -->
+	<xacro:d435_gazebo_camera parent="${parent}" prefix="${prefix}"/>
+</xacro:macro>
 </robot>

File: urdfs/sensors/vlp16.gazebo.urdf.xacro (robot description, xacro)
@@ -5,5 +5,5 @@
 			<sensor name="${link_name}_velodyne_sensor" type="ray">
 				<visualize>false</visualize>
-				<always_on>true</always_on>
+				<always_on>false</always_on>
 				<update_rate>10</update_rate>
 				<pose>0 0 0 0 0 0</pose>

Commit message: change topic name of camera form rgb to color like the one on the real camera

File: urdfs/sensors/d435_camera.gazebo.urdf.xacro (robot description, xacro)
@@ -14,10 +14,10 @@
 	    <camera name="__default__">
 		    <horizontal_fov>1.047</horizontal_fov>
-		    <image><width>1280</width><height>720</height></image>
+		    <image><width>640</width><height>480</height></image>
 		    <clip><near>0.1</near><far>100</far></clip>
 		    <noise><type>gaussian</type><mean>0.0</mean><stddev>0.007</stddev></noise>
 	    </camera>
 	    <always_on>1</always_on>
-	    <update_rate>30</update_rate>
+	    <update_rate>15</update_rate>
 	    <visualize>1</visualize>
 	    <output>points</output>
@@ -28,10 +28,10 @@
 	    <camera name="__default__">
 		    <horizontal_fov>1.047</horizontal_fov>
-		    <image><width>1280</width><height>720</height><format>L_INT8</format></image>
+		    <image><width>640</width><height>480</height><format>L_INT8</format></image>
 		    <clip><near>0.1</near><far>100</far></clip>
 		    <noise><type>gaussian</type><mean>0.0</mean><stddev>0.007</stddev></noise>
 	    </camera>
 	    <always_on>0</always_on>
-	    <update_rate>30</update_rate>
+	    <update_rate>15</update_rate>
 	    <visualize>0</visualize>
     </sensor>
@@ -41,10 +41,10 @@
 	    <camera name="__default__">
 		    <horizontal_fov>1.047</horizontal_fov>
-		    <image><width>1280</width><height>720</height><format>L_INT8</format></image>
+		    <image><width>640</width><height>480</height><format>L_INT8</format></image>
 		    <clip><near>0.1</near><far>100</far></clip>
 		    <noise><type>gaussian</type><mean>0.0</mean><stddev>0.007</stddev></noise>
 	    </camera>
 	    <always_on>0</always_on>
-	    <update_rate>30</update_rate>
+	    <update_rate>15</update_rate>
 	    <visualize>0</visualize>
     </sensor>
@@ -54,10 +54,10 @@
 	    <camera name="__default__">
 		    <horizontal_fov>1.047</horizontal_fov>
-		    <image><width>1280</width><height>720</height><format>RGB_INT8</format></image>
+		    <image><width>640</width><height>480</height><format>RGB_INT8</format></image>
 		    <clip><near>0.1</near><far>100</far></clip>
 		    <noise><type>gaussian</type><mean>0.0</mean><stddev>0.007</stddev></noise>
 	    </camera>
 	    <always_on>1</always_on>
-	    <update_rate>30</update_rate>
+	    <update_rate>15</update_rate>
 	    <visualize>1</visualize>
     </sensor>

File: urdfs/sensors/d435_camera.urdf.xacro (robot description, xacro)
@@ -50,5 +50,5 @@
 		<!-- The following are not reliable values, and should not be used for modeling -->
 		<inertial>
-			<mass value="0.564" />
+			<mass value="0.07" />
 			<origin xyz="0 0 0" />
 			<inertia ixx="0.003881243" ixy="0.0" ixz="0.0" iyy="0.000498940" iyz="0.0" izz="0.003879257" />

File: urdfs/sensors/d435_camera_openni.gazebo.urdf.xacro (robot description, xacro)
@@ -5,8 +5,8 @@
 		<sensor type="depth" name="${prefix}/camera_depth_frame_depth_sensor">
 			<always_on>true</always_on>
-			<update_rate>30.0</update_rate>
+			<update_rate>15.0</update_rate>
 			<camera name="__default__">
 				<horizontal_fov>1.482</horizontal_fov>
-				<image><format>L8</format><width>1280</width><height>720</height></image>
+				<image><format>L8</format><width>640</width><height>480</height></image>
 				<clip><near>0.1</near><far>100</far>
 				</clip>
@@ -17,6 +17,6 @@
 				<updateRate>0</updateRate>
 				<cameraName>/${prefix}/camera</cameraName>
-				<imageTopicName>/${prefix}/camera/rgb/image_raw</imageTopicName>
-				<cameraInfoTopicName>/${prefix}/camera/rgb/camera_info</cameraInfoTopicName>
+				<imageTopicName>/${prefix}/camera/color/image_raw</imageTopicName>
+				<cameraInfoTopicName>/${prefix}/camera/color/camera_info</cameraInfoTopicName>
 				<depthImageTopicName>/${prefix}/camera/depth/image_raw</depthImageTopicName>
 				<depthImageCameraInfoTopicName>/${prefix}/camera/depth/camera_info</depthImageCameraInfoTopicName>
@@ -43,8 +43,8 @@
 		<sensor type="depth" name="${prefix}/camera_depth_frame_depth_sensor">
 			<always_on>true</always_on>
-			<update_rate>30.0</update_rate>
+			<update_rate>15.0</update_rate>
 			<camera name="__default__">
 				<horizontal_fov>1.482</horizontal_fov>
-				<image><format>R8G8B8</format><width>1280</width><height>720</height></image>
+				<image><format>R8G8B8</format><width>640</width><height>480</height></image>
 				<clip><near>0.1</near><far>100</far>
 				</clip>
@@ -55,6 +55,6 @@
 				<updateRate>0</updateRate>
 				<cameraName>/${prefix}/camera</cameraName>
-				<imageTopicName>/${prefix}/camera/rgb/image_raw</imageTopicName>
-				<cameraInfoTopicName>/${prefix}/camera/rgb/camera_info</cameraInfoTopicName>
+				<imageTopicName>/${prefix}/camera/color/image_raw</imageTopicName>
+				<cameraInfoTopicName>/${prefix}/camera/color/camera_info</cameraInfoTopicName>
 				<depthImageTopicName>/${prefix}/camera/depth/image_raw</depthImageTopicName>
 				<depthImageCameraInfoTopicName>/${prefix}/camera/depth/camera_info</depthImageCameraInfoTopicName>
