Commit message: Update realsense xacros

File: urdfs/sensors/d435_camera.urdf.xacro (robot description, xacro)
@@ -2,8 +2,11 @@
 <robot xmlns:xacro="http://ros.org/wiki/xacro">
     <xacro:include filename="$(find realsense2_description)/urdf/_d435.urdf.xacro" />
-    <xacro:macro name="d435_camera" params="parent *origin">
+    <!--xacro:include filename="$(find sensors_description)/urdfs/sensors/realsense.gazebo.urdf.xacro"/-->
+    <xacro:macro name="d435_camera" params="parent prefix *origin">
 	<xacro:sensor_d435 parent="${parent}">
 	    <xacro:insert_block name="origin" />
 	</xacro:sensor_d435>
+    <!-- Gazebo multisense plugin -->
+    <!--xacro:realsense_sensor prefix="${prefix}"/-->
     </xacro:macro>
 </robot>

File: urdfs/sensors/realsense.gazebo.urdf.xacro (robot description, xacro)
@@ -2,14 +2,14 @@
 <robot xmlns:xacro="http://ros.org/wiki/xacro">
 <xacro:macro name="realsense_sensor" params="prefix">
-<gazebo>
-	<!--<plugin name="realsense_plugin" filename="libRealSensePlugin.so"/>-->
-	<plugin name="realsense_plugin" filename="librealsense_gazebo_plugin.so">
+<!--gazebo>
+    <plugin name="realsense_plugin" filename="librealsense_gazebo_plugin.so">
 		<prefix>${prefix}</prefix>
 	</plugin>
-</gazebo>
-<gazebo reference="${prefix}/${parent}_camera_joint" type="fixed">
+</gazebo-->
+<!--<plugin name="realsense_plugin" filename="libRealSensePlugin.so"/>-->
+<!--gazebo reference="${prefix}/${parent}_camera_joint" type="fixed">
 	<pose frame="">0 0 0.015 0 0 0</pose>
-</gazebo>
-<gazebo reference="${prefix}/camera_link">
+</gazebo-->
+<!--gazebo reference="${prefix}/camera_link">
 		<inertial>
 			<mass>0.0615752</mass>
@@ -73,6 +73,6 @@
 			</surface>
 		</collision>
-</gazebo>
-<gazebo reference="${prefix}/camera_fisheye_frame">
+</gazebo-->
+<!--gazebo reference="${prefix}/camera_fisheye_frame">
 		<sensor name="${prefix}color" type="camera">
 			<pose frame="">0 -0.046 0.004 0 0 0</pose>
@@ -87,6 +87,6 @@
 			<visualize>1</visualize>
 		</sensor>
-</gazebo>
-<gazebo reference="${prefix}/camera_left_ir_frame">
+</gazebo-->
+<!--gazebo reference="${prefix}/camera_left_ir_frame">
 		<sensor name="${prefix}ired1" type="camera">
 			<pose frame="">0 -0.06 0.004 0 0 0</pose>
@@ -101,6 +101,6 @@
 			<visualize>0</visualize>
 		</sensor>
-</gazebo>
-<gazebo reference="${prefix}/camera_right_ir_frame">
+</gazebo-->
+<!--gazebo reference="${prefix}/camera_right_ir_frame">
 		<sensor name="${prefix}ired2" type="camera">
 			<pose frame="">0 0.01 0.004 0 0 0</pose>
@@ -115,6 +115,6 @@
 			<visualize>0</visualize>
 		</sensor>
-</gazebo>
-<gazebo reference="${prefix}/camera_depth_frame">
+</gazebo-->
+<!--gazebo reference="${prefix}/camera_depth_frame">
 		<sensor name="${prefix}depth" type="depth">
 			<pose frame="">0 -0.03 0.004 0 0 0</pose>
@@ -129,5 +129,5 @@
 			<visualize>0</visualize>
 		</sensor>
-</gazebo>
+</gazebo-->
 </xacro:macro>
 </robot>

Commit message: Have the realsense camera use the openni driver for depth / point clouds

File: urdfs/sensors/d435_camera.urdf.xacro (robot description, xacro)
@@ -109,4 +109,5 @@
 	<!-- Gazebo realsense plugin -->
 	<xacro:d435_gazebo_camera parent="${parent}" prefix="${prefix}"/>
+	<xacro:asus_xtion_depth_sensor prefix="${prefix}"/>
 </xacro:macro>
 </robot>

File: urdfs/sensors/d435_camera_openni.gazebo.urdf.xacro (robot description, xacro)
@@ -1,4 +1,42 @@
 <?xml version="1.0"?>
 <robot xmlns:xacro="http://ros.org/wiki/xacro">
+<xacro:macro name="asus_xtion_depth_sensor" params="prefix">
+	<gazebo reference="${prefix}/camera_depth_frame">
+		<sensor type="depth" name="${prefix}/camera_depth_frame_depth_sensor">
+			<always_on>true</always_on>
+			<update_rate>60.0</update_rate>
+			<camera name="__default__">
+				<horizontal_fov>1.047</horizontal_fov>
+				<image><format>R8G8B8</format><width>640</width><height>480</height></image>
+				<clip><near>0.1</near><far>100</far>
+				</clip>
+			</camera>
+			<plugin name="${prefix}/camera_depth_frame_controller" filename="libgazebo_ros_openni_kinect.so">
+				<baseline>0.2</baseline>
+				<alwaysOn>true</alwaysOn>
+				<updateRate>0</updateRate>
+				<cameraName>/${prefix}/camera_ir</cameraName>
+				<imageTopicName>/${prefix}/camera_ir/depth/image_raw</imageTopicName>
+				<cameraInfoTopicName>/${prefix}/camera_ir/depth/camera_info</cameraInfoTopicName>
+				<depthImageTopicName>/${prefix}/camera_ir/depth/image_raw</depthImageTopicName>
+				<depthImageCameraInfoTopicName>/${prefix}/camera_ir/depth/camera_info</depthImageCameraInfoTopicName>
+				<pointCloudTopicName>/${prefix}/camera_ir/depth/points</pointCloudTopicName>
+				<frameName>${prefix}/camera_depth_optical_frame</frameName>
+				<pointCloudCutoff>0.1</pointCloudCutoff>
+				<distortionK1>0.00000001</distortionK1>
+				<distortionK2>0.00000001</distortionK2>
+				<distortionK3>0.00000001</distortionK3>
+				<distortionT1>0.00000001</distortionT1>
+				<distortionT2>0.00000001</distortionT2>
+				<CxPrime>0</CxPrime>
+				<Cx>0</Cx>
+				<Cy>0</Cy>
+				<focalLength>0</focalLength>
+				<hackBaseline>0</hackBaseline>
+			</plugin>
+		</sensor>
+		<material value="Gazebo/Red"/>
+	</gazebo>
+</xacro:macro>
 <xacro:macro name="d435_gazebo_camera" params="parent prefix">
 <gazebo>
@@ -6,50 +44,7 @@
 	<plugin name="realsense_plugin" filename="librealsense_gazebo_plugin.so">
 		<prefix>${prefix}</prefix>
-		<pointCloudTopicName>ZZZZZ</pointCloudTopicName>
-		<pointCloudCutoff>0.2</pointCloudCutoff>
 	</plugin>
 </gazebo>
-<gazebo reference="${parent}">
-    <sensor type="depth" name="${parent}_depth_sensor">
-	<always_on>true</always_on>
-	<update_rate>30.0</update_rate>
-	<camera>
-		<horizontal_fov>${58.0*PI/180.0}</horizontal_fov>
-			<image>
-				<format>L8</format>
-				<width>640</width>
-				<height>480</height>
-			</image>
-		<clip>
-			<near>0.48</near>
-			<far>3.5</far>
-		</clip>
-	</camera>
-	<plugin name="${prefix}_controller" filename="libgazebo_ros_openni_kinect.so">
-		<baseline>0.05</baseline>
-		<alwaysOn>true</alwaysOn>
-		<updateRate>30.0</updateRate>
-		<cameraName>${prefix}ired1</cameraName>
-		<imageTopicName>/${prefix}/depth/image_raw</imageTopicName>
-		<cameraInfoTopicName>/${prefix}/depth/camera_info</cameraInfoTopicName>
-		<depthImageTopicName>/${prefix}/depth/image_raw</depthImageTopicName>
-		<depthImageCameraInfoTopicName>/${prefix}/depth/camera_info</depthImageCameraInfoTopicName>
-		<pointCloudTopicName>/${prefix}/depth/points</pointCloudTopicName>
-		<frameName>${prefix}/camera_left_ir_frame</frameName>
-		<pointCloudCutoff>0.1</pointCloudCutoff>
-		<distortionK1>0.0</distortionK1>
-		<distortionK2>0.0</distortionK2>
-		<distortionK3>0.0</distortionK3>
-		<distortionT1>0.0</distortionT1>
-		<distortionT2>0.0</distortionT2>
-		<CxPrime>0</CxPrime>
-		<Cx>0</Cx>
-		<Cy>0</Cy>
-		<focalLength>0</focalLength>
-		<hackBaseline>0</hackBaseline>
-	</plugin>
-    </sensor>
-</gazebo>
-<gazebo reference="${prefix}/camera_depth_frame">
+<!--gazebo reference="${prefix}/camera_depth_frame">
     <sensor name="${prefix}depth" type="depth">
 	    <camera name="__default__">
@@ -64,5 +59,5 @@
 	    <output>points</output>
     </sensor>
-</gazebo>
+</gazebo-->
 <gazebo reference="${prefix}/camera_left_ir_frame">
     <sensor name="${prefix}ired1" type="camera">

Commit message: bug fix

File: urdfs/sensors/d435_camera.urdf.xacro (robot description, xacro)
@@ -108,6 +108,6 @@
 	<link name="${prefix}/camera_color_optical_frame"/>
 	<!-- Gazebo realsense plugin -->
-	<xacro:d435_gazebo_camera parent="${parent}" prefix="${prefix}"/>
-	<xacro:asus_xtion_depth_sensor prefix="${prefix}"/>
+	<!--xacro:d435_gazebo_camera parent="${parent}" prefix="${prefix}"/-->
+	<xacro:asus_xtion_rgb_sensor prefix="${prefix}"/>
 </xacro:macro>
 </robot>

File: urdfs/sensors/d435_camera_openni.gazebo.urdf.xacro (robot description, xacro)
@@ -5,8 +5,8 @@
 		<sensor type="depth" name="${prefix}/camera_depth_frame_depth_sensor">
 			<always_on>true</always_on>
-			<update_rate>60.0</update_rate>
+			<update_rate>30.0</update_rate>
 			<camera name="__default__">
 				<horizontal_fov>1.047</horizontal_fov>
-				<image><format>R8G8B8</format><width>640</width><height>480</height></image>
+				<image><format>L8</format><width>640</width><height>480</height></image>
 				<clip><near>0.1</near><far>100</far>
 				</clip>
@@ -16,10 +16,10 @@
 				<alwaysOn>true</alwaysOn>
 				<updateRate>0</updateRate>
-				<cameraName>/${prefix}/camera_ir</cameraName>
-				<imageTopicName>/${prefix}/camera_ir/depth/image_raw</imageTopicName>
-				<cameraInfoTopicName>/${prefix}/camera_ir/depth/camera_info</cameraInfoTopicName>
-				<depthImageTopicName>/${prefix}/camera_ir/depth/image_raw</depthImageTopicName>
-				<depthImageCameraInfoTopicName>/${prefix}/camera_ir/depth/camera_info</depthImageCameraInfoTopicName>
-				<pointCloudTopicName>/${prefix}/camera_ir/depth/points</pointCloudTopicName>
+				<cameraName>/${prefix}/camera</cameraName>
+				<imageTopicName>/${prefix}/camera/rgb/image_raw</imageTopicName>
+				<cameraInfoTopicName>/${prefix}/camera/rgb/camera_info</cameraInfoTopicName>
+				<depthImageTopicName>/${prefix}/camera/depth/image_raw</depthImageTopicName>
+				<depthImageCameraInfoTopicName>/${prefix}/camera/depth/camera_info</depthImageCameraInfoTopicName>
+				<pointCloudTopicName>/${prefix}/camera/depth/points</pointCloudTopicName>
 				<frameName>${prefix}/camera_depth_optical_frame</frameName>
 				<pointCloudCutoff>0.1</pointCloudCutoff>
@@ -39,183 +39,41 @@
 	</gazebo>
 </xacro:macro>
-<xacro:macro name="d435_gazebo_camera" params="parent prefix">
-<gazebo>
-	<!--<plugin name="realsense_plugin" filename="libRealSensePlugin.so"/>-->
-	<plugin name="realsense_plugin" filename="librealsense_gazebo_plugin.so">
-		<prefix>${prefix}</prefix>
-	</plugin>
-</gazebo>
-<!--gazebo reference="${prefix}/camera_depth_frame">
-    <sensor name="${prefix}depth" type="depth">
-	    <camera name="__default__">
-		    <horizontal_fov>1.047</horizontal_fov>
-		    <image><width>640</width><height>480</height></image>
-		    <clip><near>0.1</near><far>100</far></clip>
-		    <noise><type>gaussian</type><mean>0.0</mean><stddev>0.007</stddev></noise>
-	    </camera>
-	    <always_on>1</always_on>
-	    <update_rate>60</update_rate>
-	    <visualize>1</visualize>
-	    <output>points</output>
-    </sensor>
-</gazebo-->
-<gazebo reference="${prefix}/camera_left_ir_frame">
-    <sensor name="${prefix}ired1" type="camera">
-	    <camera name="__default__">
-		    <horizontal_fov>1.047</horizontal_fov>
-		    <image><width>640</width><height>480</height><format>L_INT8</format></image>
-		    <clip><near>0.1</near><far>100</far></clip>
-		    <noise><type>gaussian</type><mean>0.0</mean><stddev>0.007</stddev></noise>
-	    </camera>
-	    <always_on>0</always_on>
-	    <update_rate>60</update_rate>
-	    <visualize>0</visualize>
-    </sensor>
-</gazebo>
-<gazebo reference="${prefix}/camera_right_ir_frame">
-    <sensor name="${prefix}ired2" type="camera">
-	    <camera name="__default__">
-		    <horizontal_fov>1.047</horizontal_fov>
-		    <image><width>640</width><height>480</height><format>L_INT8</format></image>
-		    <clip><near>0.1</near><far>100</far></clip>
-		    <noise><type>gaussian</type><mean>0.0</mean><stddev>0.007</stddev></noise>
-	    </camera>
-	    <always_on>0</always_on>
-	    <update_rate>60</update_rate>
-	    <visualize>0</visualize>
-    </sensor>
-</gazebo>
-<gazebo reference="${prefix}/camera_color_frame">
-    <sensor name="${prefix}color" type="camera">
-	    <camera name="__default__">
-		    <horizontal_fov>1.047</horizontal_fov>
-		    <image><width>640</width><height>480</height><format>RGB_INT8</format></image>
-		    <clip><near>0.1</near><far>100</far></clip>
-		    <noise><type>gaussian</type><mean>0.0</mean><stddev>0.007</stddev></noise>
-	    </camera>
-	    <always_on>0</always_on>
-	    <update_rate>60</update_rate>
-	    <visualize>1</visualize>
-    </sensor>
-</gazebo>
-<!--gazebo reference="${prefix}/camera_link">
-		<inertial>
-			<mass>0.564</mass>
-			<inertia>
-				<ixx>0.003881243</ixx>
-				<ixy>0</ixy>
-				<ixz>0</ixz>
-				<iyy>0.000498940</iyy>
-				<iyz>0</iyz>
-				<izz>0.003879257</izz>
-			</inertia>
-			<pose frame=''>${d435_cam_mount_from_center_offset} ${-d435_cam_depth_py} 0 ${M_PI/2} 0 ${M_PI/2}</pose>
-		</inertial>
-		<self_collide>0</self_collide>
-		<enable_wind>0</enable_wind>
-		<kinematic>0</kinematic>
-		<gravity>1</gravity>
-		<visual name="visual">
-			<geometry>
-				<mesh>
-					<uri>model://realsense_camera/meshes/realsense.dae</uri>
-				</mesh>
-			</geometry>
-		</visual-->
-		<!--collision name='collision'>
-			<laser_retro>0</laser_retro>
-				<max_contacts>10</max_contacts>
-				<pose frame=''>0 ${-d435_cam_depth_py} 0 0 0 0</pose>
-				<geometry>
-					<box><size>${d435_cam_depth} ${d435_cam_width} ${d435_cam_height}</size></box>
-				</geometry>
-			<surface>
-				<friction>
-					<ode><mu>1</mu><mu2>1</mu2><fdir1>0 0 0</fdir1><slip1>0</slip1><slip2>0</slip2></ode>
-					<torsional>
-						<coefficient>1</coefficient>
-						<patch_radius>0</patch_radius>
-						<surface_radius>0</surface_radius>
-						<use_patch_radius>1</use_patch_radius>
-						<ode><slip>0</slip></ode>
-					</torsional>
-				</friction>
-				<bounce>
-					<restitution_coefficient>0</restitution_coefficient>
-					<threshold>1e+06</threshold>
-				</bounce>
-				<contact>
-					<collide_without_contact>0</collide_without_contact>
-					<collide_without_contact_bitmask>1</collide_without_contact_bitmask>
-					<collide_bitmask>1</collide_bitmask>
-					<ode><soft_cfm>0</soft_cfm><soft_erp>0.2</soft_erp><kp>1e+13</kp><kd>1</kd><max_vel>0.01</max_vel><min_depth>0</min_depth></ode>
-					<bullet>
-						<split_impulse>1</split_impulse>
-						<split_impulse_penetration_threshold>-0.01</split_impulse_penetration_threshold>
-						<soft_cfm>0</soft_cfm>
-						<soft_erp>0.2</soft_erp>
-						<kp>1e+13</kp>
-						<kd>1</kd>
-					</bullet>
-				</contact>
-			</surface>
-		</collision>
-</gazebo-->
-<!--gazebo reference="${prefix}/camera_color_frame">
-		<sensor name="${prefix}color" type="camera">
-			<pose frame=''>0 -0.046 0.004 0 0 0</pose>
+<xacro:macro name="asus_xtion_rgb_sensor" params="prefix">
+	<gazebo reference="${prefix}/camera_depth_frame">
+		<sensor type="depth" name="${prefix}/camera_depth_frame_depth_sensor">
+			<always_on>true</always_on>
+			<update_rate>30.0</update_rate>
 			<camera name="__default__">
 				<horizontal_fov>1.047</horizontal_fov>
-				<image><width>640</width><height>480</height><format>RGB_INT8</format></image>
-				<clip><near>0.1</near><far>100</far></clip>
-				<noise><type>gaussian</type><mean>0.0</mean><stddev>0.007</stddev></noise>
+				<image><format>R8G8B8</format><width>640</width><height>480</height></image>
+				<clip><near>0.1</near><far>100</far>
+				</clip>
 			</camera>
-			<always_on>0</always_on>
-			<update_rate>60</update_rate>
-			<visualize>1</visualize>
+			<plugin name="${prefix}/camera_depth_frame_controller" filename="libgazebo_ros_openni_kinect.so">
+				<baseline>0.2</baseline>
+				<alwaysOn>true</alwaysOn>
+				<updateRate>0</updateRate>
+				<cameraName>/${prefix}/camera</cameraName>
+				<imageTopicName>/${prefix}/camera/rgb/image_raw</imageTopicName>
+				<cameraInfoTopicName>/${prefix}/camera/rgb/camera_info</cameraInfoTopicName>
+				<depthImageTopicName>/${prefix}/camera/depth/image_raw</depthImageTopicName>
+				<depthImageCameraInfoTopicName>/${prefix}/camera/depth/camera_info</depthImageCameraInfoTopicName>
+				<pointCloudTopicName>/${prefix}/camera/depth/points</pointCloudTopicName>
+				<frameName>${prefix}/camera_depth_optical_frame</frameName>
+				<pointCloudCutoff>0.1</pointCloudCutoff>
+				<distortionK1>0.00000001</distortionK1>
+				<distortionK2>0.00000001</distortionK2>
+				<distortionK3>0.00000001</distortionK3>
+				<distortionT1>0.00000001</distortionT1>
+				<distortionT2>0.00000001</distortionT2>
+				<CxPrime>0</CxPrime>
+				<Cx>0</Cx>
+				<Cy>0</Cy>
+				<focalLength>0</focalLength>
+				<hackBaseline>0</hackBaseline>
+			</plugin>
 		</sensor>
-</gazebo>
-<gazebo reference="${prefix}/camera_left_ir_frame">
-		<sensor name="${prefix}ired1" type="camera">
-			<pose frame=''>0 -0.06 0.004 0 0 0</pose>
-			<camera name="__default__">
-				<horizontal_fov>1.047</horizontal_fov>
-				<image><width>640</width><height>480</height><format>L_INT8</format></image>
-				<clip><near>0.1</near><far>100</far></clip>
-				<noise><type>gaussian</type><mean>0.0</mean><stddev>0.007</stddev></noise>
-			</camera>
-			<always_on>0</always_on>
-			<update_rate>60</update_rate>
-			<visualize>0</visualize>
-		</sensor>
-</gazebo>
-<gazebo reference="${prefix}/camera_right_ir_frame">
-		<sensor name="${prefix}ired2" type="camera">
-			<pose frame=''>0 0.01 0.004 0 0 0</pose>
-			<camera name="__default__">
-				<horizontal_fov>1.047</horizontal_fov>
-				<image><width>640</width><height>480</height><format>L_INT8</format></image>
-				<clip><near>0.1</near><far>100</far></clip>
-				<noise><type>gaussian</type><mean>0.0</mean><stddev>0.007</stddev></noise>
-			</camera>
-			<always_on>0</always_on>
-			<update_rate>60</update_rate>
-			<visualize>0</visualize>
-		</sensor>
-</gazebo>
-<gazebo reference="${prefix}/camera_depth_frame">
-		<sensor name="${prefix}depth" type="depth">
-			<pose frame=''>0 -0.03 0.004 0 0 0</pose>
-			<camera name="__default__">
-				<horizontal_fov>1.047</horizontal_fov>
-				<image><width>640</width><height>480</height></image>
-				<clip><near>0.1</near><far>100</far></clip>
-				<noise><type>gaussian</type><mean>0.0</mean><stddev>0.007</stddev></noise>
-			</camera>
-			<always_on>1</always_on>
-			<update_rate>60</update_rate>
-			<visualize>0</visualize>
-		</sensor>
-</gazebo-->
+		<material value="Gazebo/Red"/>
+	</gazebo>
 </xacro:macro>
 </robot>

Commit message: changed realsense mass, it was 0.56 kg!!!!! setting to 70 grams as per datasheet

File: urdfs/sensors/d435_camera.urdf.xacro (robot description, xacro)
@@ -48,7 +48,6 @@
 			</geometry>
 		</collision>
-		<!-- The following are not reliable values, and should not be used for modeling -->
 		<inertial>
-			<mass value="0.564" />
+                        <mass value="0.07" /> <!-- check this!-->
 			<origin xyz="0 0 0" />
 			<inertia ixx="0.003881243" ixy="0.0" ixz="0.0" iyy="0.000498940" iyz="0.0" izz="0.003879257" />

Commit message: Changed origin of the D435 cameras in order to see the image properly

File: urdfs/sensors/d435_camera.urdf.xacro (robot description, xacro)
@@ -57,5 +57,5 @@
 	<!-- camera depth joints and links -->
 	<joint name="${prefix}/camera_depth_joint" type="fixed">
-		<origin xyz="0 0 0" rpy="0 0 0"/>
+		<origin xyz="0.01 0 0" rpy="0 0 0"/>
 		<parent link="${prefix}/camera_link"/>
 		<child link="${prefix}/camera_depth_frame" />
@@ -96,5 +96,5 @@
 	<!-- camera color joints and links -->
 	<joint name="${prefix}/camera_color_joint" type="fixed">
-		<origin xyz="0 ${d435_cam_depth_to_color_offset} 0" rpy="0 0 0" />
+		<origin xyz="0.01 ${d435_cam_depth_to_color_offset} 0" rpy="0 0 0" />
 		<parent link="${prefix}/camera_depth_frame" />
 		<child link="${prefix}/camera_color_frame" />

Commit message: removed camera collision

File: urdfs/sensors/d435_camera.urdf.xacro (robot description, xacro)
@@ -41,11 +41,11 @@
 			<material name="aluminum"/>
 		</visual>
-		<collision>
+		<!-- <collision> -->
 			<!--origin xyz="0.0 0.0 ${r430_cam_height/2}" rpy="0 0 0"/-->
-			<origin xyz="0 ${-d435_cam_depth_py} 0" rpy="0 0 0"/>
-			<geometry>
-				<box size="${d435_cam_depth} ${d435_cam_width} ${d435_cam_height}"/>
-			</geometry>
-		</collision>
+			<!-- <origin xyz="0 ${-d435_cam_depth_py} 0" rpy="0 0 0"/> -->
+			<!-- <geometry> -->
+				<!-- <box size="${d435_cam_depth} ${d435_cam_width} ${d435_cam_height}"/> -->
+			<!-- </geometry> -->
+		<!-- </collision> -->
 		<!-- The following are not reliable values, and should not be used for modeling -->
 		<inertial>
