Commit message: repositioning lidar

File: urdfs/sensors/vlp16_velodyne.urdf.xacro (robot description, xacro)
@@ -20,5 +20,5 @@
     </joint>
     <link name="${name}_base_link">
-      <!--<inertial>
+      <inertial>
         <mass value="0.83"/>
         <origin xyz="0 0 0.03585"/>
@@ -27,6 +27,5 @@
           izz="${0.5 * 0.83 * (0.0516*0.0516)}"/>
       </inertial>
-      -->
-      <inertial>
+      <!--inertial>
           <mass value="0.0"/>
           <origin xyz="0.0 0.0 0.0"/>
@@ -35,5 +34,6 @@
                    izz="0.0"/>
       </inertial>
-      <visual>
+      -->
+      <!--visual>
         <geometry>
           <mesh filename="package://velodyne_description/meshes/VLP16_base_1.dae" />
@@ -44,5 +44,5 @@
           <mesh filename="package://velodyne_description/meshes/VLP16_base_2.dae" />
         </geometry>
-      </visual>
+      </visual>-->
       <collision>
         <origin rpy="0 0 0" xyz="0 0 0.03585"/>
@@ -53,5 +53,5 @@
     </link>
     <joint name="${name}_base_scan_joint" type="fixed" >
-      <origin xyz="0 0 0.0377" rpy="0 0 0" />
+      <origin xyz="0.035 0 0.0377" rpy="0 0 0" />
       <parent link="${name}_base_link" />
       <child link="${name}"/>
