Commit message: [feature] Defined the imu parameters in the common.xacro file
These parameters aren't set in the call of the imu because they don't
change for the imu sensor in question

File: urdfs/common.xacro (robot description, xacro)
@@ -2,4 +2,32 @@
 <robot>
 	<property name="PI" value="3.1415926535897931"/>
+	<!-- TODO checks the imus properties -->
+	<!-- Microstrain kvh1775 IMU -->
+	<property name="kvh1775_vel_mean" value="0" />
+	<property name="kvh1775_vel_stddev" value="2e-4" />
+	<property name="kvh1775_vel_bias_mean" value="0.00087" />
+	<property name="kvh1775_vel_bias_stddev" value="0.0000008" />
+	<property name="kvh1775_acc_mean" value="0" />
+	<property name="kvh1775_acc_stddev" value="1.7e-2" />
+	<property name="kvh1775_acc_bias_mean" value="0.002" />
+	<property name="kvh1775_acc_bias_stddev" value="0.001" />
+	<!-- Microstrain 3dmgx425 IMU -->
+	<property name="3dmgx425_vel_mean" value="0" />
+	<property name="3dmgx425_vel_stddev" value="2e-4" />
+	<property name="3dmgx425_vel_bias_mean" value="0.00087" />
+	<property name="3dmgx425_vel_bias_stddev" value="0.0000008" />
+	<property name="3dmgx425_acc_mean" value="0" />
+	<property name="3dmgx425_acc_stddev" value="1.7e-2" />
+	<property name="3dmgx425_acc_bias_mean" value="0.002" />
+	<property name="3dmgx425_acc_bias_stddev" value="0.001" />
+	<!-- Microstrain 3dmgx325 IMU -->
+	<property name="3dmgx325_vel_mean" value="0" />
+	<property name="3dmgx325_vel_stddev" value="2e-4" />
+	<property name="3dmgx325_vel_bias_mean" value="0.00087" />
+	<property name="3dmgx325_vel_bias_stddev" value="0.0000008" />
+	<property name="3dmgx325_acc_mean" value="0" />
+	<property name="3dmgx325_acc_stddev" value="1.7e-2" />
+	<property name="3dmgx325_acc_bias_mean" value="0.002" />
+	<property name="3dmgx325_acc_bias_stddev" value="0.001" />
 	<!-- PTU unit -->
 	<property name="pan_velocity" value="1.0" />

File: urdfs/sensors/kvh_1775_imu.urdf.xacro (robot description, xacro)
@@ -32,8 +32,13 @@
 		<!-- IMU definition -->
 		<xacro:imu_sensor imu_name="${imu_name}" imu_topic="${imu_topic}"
-		 	update_rate="${update_rate}" rate_mean="${rate_mean}" rate_stddev="${rate_stddev}"
-		 	rate_bias_mean="${rate_bias_mean}" rate_bias_stddev="${rate_bias_stddev}"
-		 	accel_mean="${accel_mean}" accel_stddev="${accel_stddev}" accel_bias_mean="${accel_bias_mean}"
-		 	accel_bias_stddev="${accel_bias_stddev}"/>
-		</xacro:macro>
+		 	update_rate="${update_rate}"
+			rate_mean="${kvh1775_vel_mean}"
+		 	rate_stddev="${kvh1775_vel_stddev}"
+		 	rate_bias_mean="${kvh1775_vel_bias_mean}"
+		 	rate_bias_stddev="${kvh1775_vel_bias_stddev}"
+		 	accel_mean="${kvh1775_acc_mean}"
+		 	accel_stddev="${kvh1775_acc_stddev}"
+			accel_bias_mean="${kvh1775_acc_bias_mean}"
+		 	accel_bias_stddev="${kvh1775_acc_bias_stddev}"/>
+	</xacro:macro>
 </robot>

File: urdfs/sensors/microstrain_3dmgx325_imu.urdf.xacro (robot description, xacro)
@@ -28,8 +28,13 @@
 		<!-- IMU definition -->
 		<xacro:imu_sensor imu_name="${imu_name}" imu_topic="${imu_topic}"
-		 	update_rate="${update_rate}" rate_mean="${rate_mean}" rate_stddev="${rate_stddev}"
-		 	rate_bias_mean="${rate_bias_mean}" rate_bias_stddev="${rate_bias_stddev}"
-		 	accel_mean="${accel_mean}" accel_stddev="${accel_stddev}" accel_bias_mean="${accel_bias_mean}"
-		 	accel_bias_stddev="${accel_bias_stddev}"/>
+		 	update_rate="${update_rate}"
+		 	rate_mean="${3dmgx325_vel_mean}"
+		 	rate_stddev="${3dmgx325_vel_stddev}"
+		 	rate_bias_mean="${3dmgx325_vel_bias_mean}"
+		 	rate_bias_stddev="${3dmgx325_vel_bias_stddev}"
+		 	accel_mean="${3dmgx325_acc_mean}"
+		 	accel_stddev="${3dmgx325_acc_stddev}"
+			accel_bias_mean="${3dmgx325_acc_bias_mean}"
+		 	accel_bias_stddev="${3dmgx325_acc_bias_stddev}"/>
 	</xacro:macro>
 </robot>

File: urdfs/sensors/microstrain_3dmgx425_imu.urdf.xacro (robot description, xacro)
@@ -2,18 +2,7 @@
 <robot xmlns:xacro="http://ros.org/wiki/xacro">
 	<xacro:include filename="$(find sensors_description)/urdfs/sensors/imu.gazebo.xacro"/>
-<!--
-	<property name="rate_mean" value="0" />
-	<property name="rate_stddev" value="2e-4" />
-	<property name="rate_bias_mean" value="0.00087" />
-	<property name="rate_bias_stddev" value="0.0000008" />
-	<property name="accel_mean" value="0" />
-	<property name="accel_stddev" value="1.7e-2" />
-	<property name="accel_bias_mean" value="0.002" />
-	<property name="accel_bias_stddev" value="0.001" />
--->
 	<!-- ============================ IMU microstrain ============================== -->
 	<!-- The xacro macro xacro:microstrain_3dmgx425_imu: imu frame -->
-	<xacro:macro name="microstrain_3dmgx425_imu" params="parent *origin imu_name imu_topic update_rate
-		rate_mean rate_stddev rate_bias_mean rate_bias_stddev accel_mean accel_stddev accel_bias_mean accel_bias_stddev">
+	<xacro:macro name="microstrain_3dmgx425_imu" params="parent *origin imu_name imu_topic update_rate">
 		<!-- Joint -->
 		<joint name="${imu_name}_joint" type="fixed">
@@ -41,8 +30,13 @@
 		<!-- IMU Gazebo plugin definition -->
 		<xacro:imu_sensor imu_name="${imu_name}" imu_topic="${imu_topic}"
-		 	update_rate="${update_rate}" rate_mean="${rate_mean}" rate_stddev="${rate_stddev}"
-		 	rate_bias_mean="${rate_bias_mean}" rate_bias_stddev="${rate_bias_stddev}"
-		 	accel_mean="${accel_mean}" accel_stddev="${accel_stddev}" accel_bias_mean="${accel_bias_mean}"
-		 	accel_bias_stddev="${accel_bias_stddev}"/>
+		 	update_rate="${update_rate}"
+		 	rate_mean="${3dmgx425_vel_mean}"
+		 	rate_stddev="${3dmgx425_vel_stddev}"
+		 	rate_bias_mean="${3dmgx425_vel_bias_mean}"
+		 	rate_bias_stddev="${3dmgx425_vel_bias_stddev}"
+		 	accel_mean="${3dmgx425_acc_mean}"
+		 	accel_stddev="${3dmgx425_acc_stddev}"
+			accel_bias_mean="${3dmgx425_acc_bias_mean}"
+		 	accel_bias_stddev="${3dmgx425_acc_bias_stddev}"/>
 	</xacro:macro>
 </robot>

Commit message: New xacro (kinetic)

File: urdfs/common.xacro (robot description, xacro)
@@ -1,71 +1,71 @@
 <?xml version="1.0"?>
-<robot>
-	<property name="PI" value="3.1415926535897931"/>
+<robot xmlns:xacro="http://ros.org/wiki/xacro">
+	<xacro:property name="PI" value="3.1415926535897931"/>
 	<!-- TODO checks the imu properties -->
 	<!-- Microstrain kvh1775 IMU -->
-	<property name="kvh_1775_vel_mean" value="0" />
-	<property name="kvh_1775_vel_stddev" value="2e-4" />
-	<property name="kvh_1775_vel_bias_mean" value="0.00087" />
-	<property name="kvh_1775_vel_bias_stddev" value="0.0000008" />
-	<property name="kvh_1775_acc_mean" value="0" />
-	<property name="kvh_1775_acc_stddev" value="1.7e-2" />
-	<property name="kvh_1775_acc_bias_mean" value="0.002" />
-	<property name="kvh_1775_acc_bias_stddev" value="0.001" />
+	<xacro:property name="kvh_1775_vel_mean" value="0" />
+	<xacro:property name="kvh_1775_vel_stddev" value="2e-4" />
+	<xacro:property name="kvh_1775_vel_bias_mean" value="0.00087" />
+	<xacro:property name="kvh_1775_vel_bias_stddev" value="0.0000008" />
+	<xacro:property name="kvh_1775_acc_mean" value="0" />
+	<xacro:property name="kvh_1775_acc_stddev" value="1.7e-2" />
+	<xacro:property name="kvh_1775_acc_bias_mean" value="0.002" />
+	<xacro:property name="kvh_1775_acc_bias_stddev" value="0.001" />
 	<!-- Microstrain 3dmgx425 IMU -->
-	<property name="microstrain_gx425_vel_mean" value="0" />
-	<property name="microstrain_gx425_vel_stddev" value="2e-4" />
-	<property name="microstrain_gx425_vel_bias_mean" value="0.00087" />
-	<property name="microstrain_gx425_vel_bias_stddev" value="0.0000008" />
-	<property name="microstrain_gx425_acc_mean" value="0" />
-	<property name="microstrain_gx425_acc_stddev" value="1.7e-2" />
-	<property name="microstrain_gx425_acc_bias_mean" value="0.002" />
-	<property name="microstrain_gx425_acc_bias_stddev" value="0.001" />
+	<xacro:property name="microstrain_gx425_vel_mean" value="0" />
+	<xacro:property name="microstrain_gx425_vel_stddev" value="2e-4" />
+	<xacro:property name="microstrain_gx425_vel_bias_mean" value="0.00087" />
+	<xacro:property name="microstrain_gx425_vel_bias_stddev" value="0.0000008" />
+	<xacro:property name="microstrain_gx425_acc_mean" value="0" />
+	<xacro:property name="microstrain_gx425_acc_stddev" value="1.7e-2" />
+	<xacro:property name="microstrain_gx425_acc_bias_mean" value="0.002" />
+	<xacro:property name="microstrain_gx425_acc_bias_stddev" value="0.001" />
 	<!-- Microstrain 3dmgx325 IMU -->
-	<property name="microstrain_gx325_vel_mean" value="0" />
-	<property name="microstrain_gx325_vel_stddev" value="2e-4" />
-	<property name="microstrain_gx325_vel_bias_mean" value="0.00087" />
-	<property name="microstrain_gx325_vel_bias_stddev" value="0.0000008" />
-	<property name="microstrain_gx325_acc_mean" value="0" />
-	<property name="microstrain_gx325_acc_stddev" value="1.7e-2" />
-	<property name="microstrain_gx325_acc_bias_mean" value="0.002" />
-	<property name="microstrain_gx325_acc_bias_stddev" value="0.001" />
+	<xacro:property name="microstrain_gx325_vel_mean" value="0" />
+	<xacro:property name="microstrain_gx325_vel_stddev" value="2e-4" />
+	<xacro:property name="microstrain_gx325_vel_bias_mean" value="0.00087" />
+	<xacro:property name="microstrain_gx325_vel_bias_stddev" value="0.0000008" />
+	<xacro:property name="microstrain_gx325_acc_mean" value="0" />
+	<xacro:property name="microstrain_gx325_acc_stddev" value="1.7e-2" />
+	<xacro:property name="microstrain_gx325_acc_bias_mean" value="0.002" />
+	<xacro:property name="microstrain_gx325_acc_bias_stddev" value="0.001" />
 	<!-- PTU unit -->
-	<property name="pan_velocity" value="1.0" />
-	<property name="pan_range" value="2.775" />
-	<property name="tilt_velocity" value="1.0" />
-	<property name="tilt_up_range" value="0.52" />
-	<property name="tilt_down_range" value="0.82" />
-	<property name="joint_effort" value="30" />
+	<xacro:property name="pan_velocity" value="1.0" />
+	<xacro:property name="pan_range" value="2.775" />
+	<xacro:property name="tilt_velocity" value="1.0" />
+	<xacro:property name="tilt_up_range" value="0.52" />
+	<xacro:property name="tilt_down_range" value="0.82" />
+	<xacro:property name="joint_effort" value="30" />
 	<!-- Asus Xtion Camera Location (Nominally 0) -->
-	<property name="asus_xtion_x" value="0.009"/>
-	<property name="asus_xtion_depth_y" value="0.045"/>
-	<property name="asus_xtion_rgb_y" value="0.01875"/>
-	<property name="asus_xtion_z" value="0.035"/>
-	<property name="asus_xtion_roll" value="${-PI/2}"/>
-	<property name="asus_xtion_pitch" value="0.0"/>
-	<property name="asus_xtion_yaw" value="${-PI/2}"/>
+	<xacro:property name="asus_xtion_x" value="0.009"/>
+	<xacro:property name="asus_xtion_depth_y" value="0.045"/>
+	<xacro:property name="asus_xtion_rgb_y" value="0.01875"/>
+	<xacro:property name="asus_xtion_z" value="0.035"/>
+	<xacro:property name="asus_xtion_roll" value="${-PI/2}"/>
+	<xacro:property name="asus_xtion_pitch" value="0.0"/>
+	<xacro:property name="asus_xtion_yaw" value="${-PI/2}"/>
 	<!-- Kinect Camera Location (Nominally 0) -->
-	<property name="kinect_x" value="0.025"/>
-	<property name="kinect_ir_y" value="0.01"/>
-	<property name="kinect_rgb_y" value="0.015"/>
-	<property name="kinect_z" value="0.052"/>
-	<property name="kinect_roll" value="${-PI/2}"/>
-	<property name="kinect_pitch" value="0.0"/>
-	<property name="kinect_yaw" value="${-PI/2}"/>
+	<xacro:property name="kinect_x" value="0.025"/>
+	<xacro:property name="kinect_ir_y" value="0.01"/>
+	<xacro:property name="kinect_rgb_y" value="0.015"/>
+	<xacro:property name="kinect_z" value="0.052"/>
+	<xacro:property name="kinect_roll" value="${-PI/2}"/>
+	<xacro:property name="kinect_pitch" value="0.0"/>
+	<xacro:property name="kinect_yaw" value="${-PI/2}"/>
 	<!-- Bumblebee mass and lengths for computing inertia tensor -->
-	<property name="b2mass" value="0.342"/>
-	<property name="b2lx" value="0.157"/>
-	<property name="b2ly" value="0.036"/>
-	<property name="b2lz" value="0.0474"/>
+	<xacro:property name="b2mass" value="0.342"/>
+	<xacro:property name="b2lx" value="0.157"/>
+	<xacro:property name="b2ly" value="0.036"/>
+	<xacro:property name="b2lz" value="0.0474"/>
 	<!-- Velodyne Lidar Location (Nominally 0) -->
-	<property name="velodyne_x" value="0.0"/>
-	<property name="velodyne_y" value="0.0"/>
-	<property name="velodyne_z" value="0.09"/>
+	<xacro:property name="velodyne_x" value="0.0"/>
+	<xacro:property name="velodyne_y" value="0.0"/>
+	<xacro:property name="velodyne_z" value="0.09"/>
 	<!-- HighDef Camera Location (Nominally 0) -->
-	<property name="cal_high_def_x" value="0.0" />
-	<property name="cal_high_def_y" value="0.0" />
-	<property name="cal_high_def_z" value="0.0" />
-	<property name="cal_high_def_roll" value="0.0" />
-	<property name="cal_high_def_pitch" value="0.0" />
-	<property name="cal_high_def_yaw" value="0.0" />
+	<xacro:property name="cal_high_def_x" value="0.0" />
+	<xacro:property name="cal_high_def_y" value="0.0" />
+	<xacro:property name="cal_high_def_z" value="0.0" />
+	<xacro:property name="cal_high_def_roll" value="0.0" />
+	<xacro:property name="cal_high_def_pitch" value="0.0" />
+	<xacro:property name="cal_high_def_yaw" value="0.0" />
 </robot>

File: urdfs/sensors/asus_xtion.urdf.xacro (robot description, xacro)
@@ -1,4 +1,4 @@
 <?xml version="1.0"?>
-<root xmlns:xacro="http://www.ros.org/wiki/xacro">
+<root xmlns:xacro="http://ros.org/wiki/xacro">
 	<xacro:include filename="$(find sensors_description)/urdfs/sensors/asus_xtion.gazebo.xacro" />
 	<!-- ===================================== ASUS & PROSILICA ==================================== -->
@@ -7,5 +7,5 @@
 		<!-- Joints -->
 		<joint name="${name}_joint" type="fixed">
-			<insert_block name="origin"/>
+			<xacro:insert_block name="origin"/>
 			<parent link="${parent}"/>
 			<child link="${name}_mount_link"/>

File: urdfs/sensors/bumblebee.urdf.xacro (robot description, xacro)
@@ -1,4 +1,4 @@
 <?xml version="1.0"?>
-<robot xmlns:xacro="http://www.ros.org/wiki/xacro">
+<robot xmlns:xacro="http://ros.org/wiki/xacro">
 	<xacro:include filename="$(find sensors_description)/urdfs/sensors/stereo_camera.gazebo.xacro"/>
 	<!-- ================================ Bumblebee ============================== -->

File: urdfs/sensors/hokuyo_laser.urdf.xacro (robot description, xacro)
@@ -6,5 +6,5 @@
 		<joint name="${name}_joint" type="fixed">
 			<axis xyz="0 0 0" />
-			<insert_block name="origin" />
+			<xacro:insert_block name="origin" />
 			<parent link="${parent}"/>
 			<child link="${name}_mount_link"/>

File: urdfs/sensors/kinect.urdf.xacro (robot description, xacro)
@@ -1,6 +1,6 @@
 <?xml version="1.0"?>
-<root xmlns:xacro="http://www.ros.org/wiki/xacro">
+<root xmlns:xacro="http://ros.org/wiki/xacro">
 	<xacro:include filename="$(find sensors_description)/urdfs/sensors/kinect.gazebo.xacro" />
-	<property name="ir_depth_rgb_offset_y" value="0.01"/> <!-- FIXME: what is this offset? -->
+	<xacro:property name="ir_depth_rgb_offset_y" value="0.01"/> <!-- FIXME: what is this offset? -->
 	<!-- ===================================== KINECT & PROSILICA ==================================== -->
 	<!-- The xacro macro xacro:kinect_prosilica_camera_swept_back contains: kinect and prosilica combo -->
@@ -8,5 +8,5 @@
 		<!-- Joints -->
 		<joint name="${name}_kinect_joint" type="fixed">
-			<insert_block name="origin"/>
+			<xacro:insert_block name="origin"/>
 			<parent link="${parent}"/>
 			<child link="${name}_kinect_link"/>

File: urdfs/sensors/kvh_1775_imu.urdf.xacro (robot description, xacro)
@@ -7,5 +7,5 @@
 		<!-- Joint -->
 		<joint name="${imu_name}_joint" type="fixed">
-			<insert_block name="origin"/>
+			<xacro:insert_block name="origin"/>
 			<parent link="${parent}" />
 			<child link="${imu_name}"/>

File: urdfs/sensors/microstrain_3dmgx325_imu.urdf.xacro (robot description, xacro)
@@ -7,5 +7,5 @@
 		<!-- Joint -->
 		<joint name="${imu_name}_joint" type="fixed">
-			<insert_block name="origin"/>
+			<xacro:insert_block name="origin"/>
 			<parent link="${parent}" />
 			<child link="${imu_name}"/>

File: urdfs/sensors/microstrain_3dmgx425_imu.urdf.xacro (robot description, xacro)
@@ -2,4 +2,5 @@
 <robot xmlns:xacro="http://ros.org/wiki/xacro">
 	<xacro:include filename="$(find sensors_description)/urdfs/sensors/imu.gazebo.xacro"/>
+<xacro:include filename="$(find sensors_description)/urdfs/common.xacro"/>
 	<!-- ============================ IMU microstrain ============================== -->
 	<!-- The xacro macro xacro:microstrain_3dmgx425_imu: imu frame -->
@@ -7,5 +8,5 @@
 		<!-- Joint -->
 		<joint name="${imu_name}_joint" type="fixed">
-			<insert_block name="origin"/>
+			<xacro:insert_block name="origin"/>
 			<parent link="${parent}" />
 			<child link="${imu_name}"/>
@@ -37,6 +38,6 @@
 		 	accel_mean="${microstrain_gx425_acc_mean}"
 		 	accel_stddev="${microstrain_gx425_acc_stddev}"
-			accel_bias_mean="${microstrain_gx425_acc_bias_mean}"
-		 	accel_bias_stddev="${microstrain_gx425_acc_bias_stddev}"/>
+			accel_bias_mean="0.002"
+		 	accel_bias_stddev="0.001"/>
 	</xacro:macro>
 </robot>

File: urdfs/sensors/multisense_sl.urdf.xacro (robot description, xacro)
@@ -4,5 +4,5 @@
 <xacro:macro name="multisense_sl" params="parent *origin prefix" >
 	<joint name="${parent}_head_root_joint" type="fixed">
-		<insert_block name="origin"/>
+		<xacro:insert_block name="origin"/>
 		<parent link="${parent}"/>
 		<child link="head_root"/>

File: urdfs/sensors/ptu_d46.transmission.xacro (robot description, xacro)
@@ -1,4 +1,4 @@
 <?xml version="1.0"?>
-<robot xmlns:xacro="http://www.ros.org/wiki/xacro">
+<robot xmlns:xacro="http://ros.org/wiki/xacro">
 	<xacro:macro name="ptu_transmission" params="name">
     	<!-- Pan assembly -->

File: urdfs/sensors/ptu_d46.urdf.xacro (robot description, xacro)
@@ -1,4 +1,4 @@
 <?xml version="1.0"?>
-<robot xmlns:xacro="http://www.ros.org/wiki/xacro">
+<robot xmlns:xacro="http://ros.org/wiki/xacro">
 	<!-- Things that are needed only for Gazebo (not the physical robot). These include sensor and controller plugin specifications -->
 	<xacro:include filename="$(find sensors_description)/urdfs/sensors/ptu_d46.transmission.xacro"/>
@@ -57,5 +57,5 @@
 		<!-- Joints -->
 		<joint name="${name}_joint" type="fixed">
-			<insert_block name="origin"/>
+			<xacro:insert_block name="origin"/>
 			<parent link="${parent}"/>
 			<child link="${name}_base_link"/>

File: urdfs/sensors/stereo_camera.gazebo.xacro (robot description, xacro)
@@ -1,4 +1,4 @@
 <?xml version="1.0"?>
-<robot xmlns:xacro="http://www.ros.org/wiki/xacro">
+<robot xmlns:xacro="http://ros.org/wiki/xacro">
 	<xacro:macro name="stereo_camera" params="reference ns frame_id update_rate baseline hfov width height format near far">
 		<gazebo reference="${reference}">

File: urdfs/sensors/velodyne.urdf.xacro (robot description, xacro)
@@ -1,4 +1,4 @@
 <?xml version="1.0"?>
-<robot xmlns:xacro="http://www.ros.org/wiki/xacro">
+<robot xmlns:xacro="http://ros.org/wiki/xacro">
 	<xacro:include filename="$(find sensors_description)/urdfs/sensors/velodyne.gazebo.xacro" />
 	<!-- ===================================== VELODYNE ==================================== -->
@@ -7,5 +7,5 @@
 		<!-- Joints -->
 		<joint name="${name}_joint" type="fixed">
-			<insert_block name="origin"/>
+			<xacro:insert_block name="origin"/>
 			<parent link="${parent}"/>
 			<child link="${name}_mount_link"/>

File: urdfs/sensors/vicon.urdf.xacro (robot description, xacro)
@@ -1,4 +1,4 @@
 <?xml version="1.0"?>
-<robot xmlns:xacro="http://www.ros.org/wiki/xacro">
+<robot xmlns:xacro="http://ros.org/wiki/xacro">
 	<!-- ======================================= VICON MARKER ====================================== -->
 	<!-- The xacro macro xacro:vicon_marker contains: vicon marker link -->
@@ -6,5 +6,5 @@
 		<!-- Joints -->
 		<joint name="vicon_maker_joint" type="floating">
-			<insert_block name="origin"/>
+			<xacro:insert_block name="origin"/>
 			<parent link="vicon_marker_link"/>
 			<child link="${child}"/>

File: urdfs/sensors/vislab_3dve.urdf.xacro (robot description, xacro)
@@ -1,4 +1,4 @@
 <?xml version="1.0"?>
-<robot xmlns:xacro="http://www.ros.org/wiki/xacro">
+<robot xmlns:xacro="http://ros.org/wiki/xacro">
 	<xacro:include filename="$(find sensors_description)/urdfs/sensors/stereo_camera.gazebo.xacro"/>
 	<xacro:macro name="vislab_3dve" params="name parent xyz rpy high_res hfov">
